File: 6502gpu.kicad_pcb (KiCad board)
At the start: 2 copper layers, 89 parts, among them J1 Conn_01x02, J2 Conn_01x08, J3 Conn_01x02, J4 Conn_01x16, J5 Conn_01x01, J6 Conn_01x03, J7 DE15_Receptacle_HighDensity, J8 Conn_01x02, J9 Conn_01x02, U1 74HC86, U10 74AHC30, U11 74AHC30, U12 74AHC30, U13 74AHC30, U14 74LV163, U15 74LV04, U16 74AC109, U17 74LV163, U18 74LV04, U19 74LV08, U2 74HC00, U20 74LV163, U21 74AHC30, U22 74AHC30, U23 74AHC30, U24 74AHC30, U25 74AC109, U26 74LV163, U27 74LV163, U28 74LV163, U29 74HC377, U3 74LV27, U30 74LV32, U31 74LV32, U32 74LV08, U33 74LV08, U4 74HC00, U5 74CBT16390, U6 74CBT16390, U7 AS7C256A-10, U8 AS7C256A-10, U9 74CBT16390, X1 25.175MHz

Commit message: Work on layout/routing
Parts:
- moved U9 185.8 mm to (62.3, 67.8)
- moved U5 182.2 mm to (43.3, 40.6)
- moved U7 170.3 mm to (59.1, 35.3), turned to 180 degrees
- moved U8 170.0 mm to (59.1, 47.6), turned to 180 degrees
- moved U6 161.0 mm to (74.9, 40.6)
- moved U33 122.1 mm to (111.7, 131.4)
- moved U32 120.2 mm to (111.8, 144.1)
- moved U31 114.2 mm to (103.5, 131.4)
- moved U30 112.9 mm to (103.4, 144.1)
- moved U28 101.2 mm to (116.3, 66.5)
- moved R9 99.2 mm to (121.6, 153.0), turned to 180 degrees
- moved R1 96.8 mm to (121.6, 150.5)
- moved R10 93.4 mm to (121.6, 145.4), turned to 180 degrees
- moved R2 93.3 mm to (121.6, 148.0)
- moved R7 90.9 mm to (121.6, 130.2)
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Connections:
- net /AddrSelect renamed /AddrSel
- net /~{CpuWe} renamed /R~{W}
- J1 pad 1: /~{CpuClock} -> /Phi2
- U1 pad 5: /~{CpuClock} -> /Phi2
- U1 pad 6: /ConfigReg/Clock -> /~{Phi2}
- U1 pad 8: /WriteMem -> /~{WriteReg}
- U29 pad 11: /ConfigReg/Clock -> /~{Phi2}
- U3 pad 4: /~{CpuClock} -> /~{Phi2}
- U3 pad 6: Net-(U1-Pad10) -> /WriteMem
- U3 pad 8: /~{WriteReg} -> Net-(U1-Pad10)
- U30 pad 1: /DAC/PixelOut0 -> /DAC/PixelOut2
- U30 pad 9: /DAC/PixelOut2 -> /DAC/PixelOut0
- U31 pad 1: /DAC/PixelOut4 -> /DAC/PixelOut6
- U31 pad 9: /DAC/PixelOut6 -> /DAC/PixelOut4
- U32 pad 1: Net-(U30-Pad3) -> Net-(U30-Pad11)
- U32 pad 11: Net-(R4-Pad1) -> Net-(R3-Pad1)
- U32 pad 12: Net-(U30-Pad11) -> Net-(U30-Pad3)
- U32 pad 3: Net-(R1-Pad1) -> Net-(R4-Pad1)
- U32 pad 4: Net-(U30-Pad6) -> Net-(U30-Pad8)
- U32 pad 6: Net-(R2-Pad1) -> Net-(R1-Pad1)
- U32 pad 8: Net-(R3-Pad1) -> Net-(R2-Pad1)
- U32 pad 9: Net-(U30-Pad8) -> Net-(U30-Pad6)
- U33 pad 1: Net-(U31-Pad3) -> Net-(U31-Pad11)
- U33 pad 11: Net-(R8-Pad1) -> Net-(R7-Pad1)
- U33 pad 12: Net-(U31-Pad11) -> Net-(U31-Pad3)
- U33 pad 3: Net-(R5-Pad1) -> Net-(R8-Pad1)
- U33 pad 4: Net-(U31-Pad6) -> Net-(U31-Pad8)
- U33 pad 6: Net-(R6-Pad1) -> Net-(R5-Pad1)
- U33 pad 8: Net-(R7-Pad1) -> Net-(R6-Pad1)
- U33 pad 9: Net-(U31-Pad8) -> Net-(U31-Pad6)
Routing:
- net /Counters/PxClock: track 0.00 -> 60.7 mm
- net /DAC/~{BlankBlack}: track 0.00 -> 43.0 mm, vias 0 -> 2
- net Net-(U26-TC): track 0.00 -> 40.4 mm, vias 0 -> 3
- net Net-(U14-TC): track 0.00 -> 40.4 mm, vias 0 -> 3
- net /Counters/~{VBlankClear}: track 0.00 -> 31.1 mm
- net /Counters/~{HBlankClear}: track 0.00 -> 31.1 mm
- net Net-(U27-TC): track 0.00 -> 21.7 mm
- net Net-(U17-TC): track 0.00 -> 21.7 mm
- net /DAC/Blue: track 0.00 -> 17.0 mm
- net /DAC/Red: track 0.00 -> 16.8 mm
- net /DAC/Green: track 0.00 -> 16.7 mm
- net Net-(U30-Pad3): track 0.00 -> 13.3 mm, vias 0 -> 2
- net Net-(U30-Pad6): track 0.00 -> 13.3 mm, vias 0 -> 2
- net Net-(U31-Pad6): track 0.00 -> 13.1 mm, vias 0 -> 2
- net Net-(U31-Pad3): track 0.00 -> 13.1 mm, vias 0 -> 2
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Other:
- copper layers 2 -> 4
- board text added: "+5V"
- board text added: "Blank Black"
- board text added: "Blank White"
- board text added: "Counters"
- board text added: "D0"
- board text added: "D1"
- board text added: "D2"
- board text added: "D3"
- board text added: "D4"
- board text added: "D5"
- board text added: "D6"
- board text added: "D7"
- board text added: "DAC"
- board text added: "GND"
- board text added: "Pixel Clock"
- board text added: "VRAM"

Commit message: More routing work
Parts:
- moved C35 179.8 mm to (39.6, 109.2)
- moved C14 151.4 mm to (99.1, 39.4), turned to -90 degrees
- moved C17 148.6 mm to (99.1, 53.3), turned to -90 degrees
- moved C20 148.0 mm to (99.1, 66.7), turned to -90 degrees
- moved C30 122.9 mm to (103.5, 151.8)
- moved C32 112.4 mm to (111.8, 151.8)
- moved C31 111.3 mm to (103.5, 123.8)
- moved C33 101.8 mm to (111.8, 123.8)
- moved C34 81.2 mm to (222.9, 26.0), turned to -90 degrees
- moved C1 76.2 mm to (159.5, 99.6)
- moved C26 75.3 mm to (114.3, 39.4), turned to -90 degrees
- moved C27 73.5 mm to (114.3, 53.3), turned to -90 degrees
- moved C28 73.2 mm to (114.3, 66.7), turned to -90 degrees
- moved C2 67.2 mm to (167.6, 98.0)
- moved C3 58.6 mm to (175.7, 98.0)
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Other:
- board text added: "Column"
- board text added: "Row"

Commit message: pcb organization
Parts:
- added J10: Conn_01x10, Connector_PinHeader_2.54mm:PinHeader_1x10_P2.54mm_Vertical, F.Cu at (114.3, 36.8)
- added J11: Conn_01x03, Connector_PinHeader_2.54mm:PinHeader_1x03_P2.54mm_Vertical, F.Cu at (127.6, 137.2)
- added J12: Conn_01x03, Connector_PinHeader_2.54mm:PinHeader_1x03_P2.54mm_Vertical, F.Cu at (144.8, 136.5)
- added J13: Conn_01x03, Connector_PinHeader_2.54mm:PinHeader_1x03_P2.54mm_Vertical, F.Cu at (156.2, 137.2)
- added J14: Conn_01x03, Connector_PinHeader_2.54mm:PinHeader_1x03_P2.54mm_Vertical, F.Cu at (172.1, 136.5)
- added J15: Conn_01x03, Connector_PinHeader_2.54mm:PinHeader_1x03_P2.54mm_Vertical, F.Cu at (86.4, 155.6)
- added J16: Conn_01x01, Connector_PinHeader_2.54mm:PinHeader_1x01_P2.54mm_Vertical, F.Cu at (241.3, 22.2)
- J5: value Conn_01x01 -> Conn_01x02; footprint Connector_PinHeader_2.54mm:PinHeader_1x01_P2.54mm_Vertical -> Connector_PinHeader_2.54mm:PinHeader_1x02_P2.54mm_Vertical
- J8: value Conn_01x02 -> Conn_01x08; footprint Connector_PinHeader_2.54mm:PinHeader_1x02_P2.54mm_Vertical -> Connector_PinHeader_2.54mm:PinHeader_1x08_P2.54mm_Vertical
- J9: value Conn_01x02 -> Conn_01x10; footprint Connector_PinHeader_2.54mm:PinHeader_1x02_P2.54mm_Vertical -> Connector_PinHeader_2.54mm:PinHeader_1x10_P2.54mm_Vertical
- moved C5 194.6 mm to (43.2, 51.4)
- moved C7 185.8 mm to (47.6, 90.8)
- moved C9 184.1 mm to (55.2, 74.3)
- moved C6 176.3 mm to (57.1, 87.0)
- moved C8 176.3 mm to (57.1, 94.0)
- moved J6 115.1 mm to (67.9, 102.2)
- moved C16 108.2 mm to (154.9, 35.6)
- moved J9 102.8 mm to (137.8, 36.8)
- moved J8 97.9 mm to (139.1, 150.5)
- moved C10 89.9 mm to (154.9, 52.1)
- moved C15 89.5 mm to (154.9, 69.8)
- moved C22 86.5 mm to (154.9, 86.4)
- moved C11 83.0 mm to (163.8, 52.1)
- moved C18 82.5 mm to (163.8, 69.8)
- moved C12 76.6 mm to (172.7, 52.1)
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Connections:
- net /Counters/HBlank renamed /HBlank
- net /Counters/VBlank renamed /VBlank
- net /DAC/Blue renamed /Blue
- net /DAC/Green renamed /Green
- net /DAC/Red renamed /Red
- J7 pad 13: Net-(J9-Pin_2) -> /~{HSync}
- J7 pad 14: Net-(J8-Pin_2) -> /~{VSync}
- J8 pad 1: /~{VSync} -> /DAC/PixelOut0
- J8 pad 2: Net-(J8-Pin_2) -> /DAC/PixelOut1
- J9 pad 1: /~{HSync} -> /Counters/Row0
- J9 pad 2: Net-(J9-Pin_2) -> /Counters/Row1
- U2 pad 6: /~{EnableCPU} -> /~{FbSelected}
- U3 pad 3: /~{EnableCPU} -> /~{FbSelected}
- U3 pad 9: /~{EnableCPU} -> /~{FbSelected}
Routing:
- net +5V: track 0.00 -> 52.9 mm, vias 0 -> 27
- net /ConfigReg/BlankWhite: track 0.00 -> 27.4 mm
- net /Blue: track 17.0 -> 42.6 mm
- net GND: track 0.00 -> 18.7 mm, vias 0 -> 6
- net /Green: track 16.7 -> 34.7 mm
- net /Counters/Row8: track 0.00 -> 10.2 mm
- net /Counters/Col8: track 0.00 -> 10.2 mm
- net /Red: track 16.8 -> 26.6 mm
- net /Counters/Col9: track 0.00 -> 9.11 mm
- net /Counters/Row9: track 0.00 -> 8.96 mm
- net /Counters/Row3: track 0.00 -> 7.36 mm
- net /Counters/Row4: track 0.00 -> 7.36 mm
- net /Counters/Col3: track 0.00 -> 7.36 mm
- net /Counters/Col4: track 0.00 -> 7.36 mm
- net /Counters/Row5: track 0.00 -> 6.83 mm
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- added copper zone on In1.Cu, net +5V
- added copper zone on B.Cu, net GND
- added copper zone on F.Cu, net GND
- added copper zone on In2.Cu, net GND
Other:
- board text added: "$4000-$7FFF"
- board text added: "$8000-$BFFF"
- board text added: "Address Select"
- board text added: "Analog 75Ω Color"
- board text added: "B0"
- board text added: "B1"
- board text added: "Blue"
- board text added: "C0"
- board text added: "C1"
- board text added: "C2"
- board text added: "C3"
- board text added: "C4"
- board text added: "C5"
- board text added: "C6"
- board text added: "C7"
- board text added: "C8"
- board text added: "C9"
- board text added: "Clear"
- board text added: "Column Counter"
- board text added: "Digital Color"
- board text added: "G0"
- board text added: "G1"
- board text added: "G2"
- board text added: "Green"
- board text added: "HBlank"
- board text added: "Jumper"
- board text added: "R0"
- board text added: "R1"
- board text added: "R2"
- board text added: "R3"
- board text added: "R4"
- board text added: "R5"
- board text added: "R6"
- board text added: "R7"
- board text added: "R8"
- board text added: "R9"
- board text added: "Red"
- board text added: "Row Counter"
- board text added: "R~{W}"
- board text added: "Set"
- board text added: "VBlank"
- board text added: "~{Clear}"
- board text added: "~{FbSel}"
- board text added: "~{HSync}"
- board text added: "~{Set}"
- board text added: "~{VSync}"
- board text removed: "~{WE}"

Commit message: Suuuper dense routing for column counter
Parts:
- U16, U25: value 74AC109 -> 74HC109
- moved J13 225.5 mm to (-67.9, 113.0)
- moved J14 225.5 mm to (-52.1, 112.4)
- moved J8 225.5 mm to (-85.1, 126.4)
- moved C30 192.9 mm to (248.9, 123.2), turned to 90 degrees
- moved C32 187.9 mm to (248.9, 114.3), turned to 90 degrees
- moved R9 184.3 mm to (249.6, 104.8), turned to -90 degrees
- moved U30 182.3 mm to (240.7, 123.2), turned to 90 degrees
- moved R1 180.9 mm to (247.0, 104.8), turned to 90 degrees
- moved R2 177.5 mm to (244.5, 104.8), turned to 90 degrees
- moved U32 177.1 mm to (240.7, 114.3), turned to 90 degrees
- moved R10 174.1 mm to (241.9, 104.8), turned to -90 degrees
- moved R3 170.7 mm to (239.4, 104.8), turned to 90 degrees
- moved R4 167.3 mm to (236.9, 104.8), turned to 90 degrees
- moved U31 166.4 mm to (228.0, 123.2), turned to 90 degrees
- moved R5 163.9 mm to (234.3, 104.8), turned to 90 degrees
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Connections:
- U10 pad 11: /Counters/Col6 -> /Counters/Col9
- U10 pad 12: /Counters/Col9 -> /Counters/Col6
- U15 pad 1: /Counters/Col5 -> GND
- U15 pad 10: unconnected-(U15-Pad10) -> /Counters/~{Col6}
- U15 pad 11: GND -> /Counters/Col6
- U15 pad 12: /Counters/VBlankSet -> /Counters/~{Col5}
- U15 pad 13: Net-(U15-Pad13) -> /Counters/Col5
- U15 pad 2: /Counters/~{Col5} -> unconnected-(U15-Pad2)
- U15 pad 3: /Counters/Col6 -> GND
- U15 pad 4: /Counters/~{Col6} -> unconnected-(U15-Pad4)
- U18 pad 10: unconnected-(U18-Pad10) -> /Counters/VBlankSet
- U18 pad 11: GND -> Net-(U18-Pad11)
- U21 pad 8: Net-(U15-Pad13) -> Net-(U18-Pad11)
Routing:
- net /Counters/Col9: track 9.11 -> 92.3 mm, vias 0 -> 4
- net /Counters/Col7: track 5.78 -> 66.7 mm, vias 0 -> 2
- net /Counters/Col6: track 6.31 -> 64.2 mm, vias 0 -> 3
- net /Counters/Col5: track 6.83 -> 62.0 mm, vias 0 -> 3
- net /Counters/Col3: track 7.36 -> 58.6 mm, vias 0 -> 4
- net /Counters/Col2: track 6.83 -> 57.7 mm, vias 0 -> 4
- net /Counters/Col1: track 6.31 -> 56.6 mm, vias 0 -> 4
- net /Counters/Col0: track 5.78 -> 55.6 mm, vias 0 -> 4
- net +5V: track 52.9 -> 80.7 mm, vias 27 -> 42
- net /Counters/Col8: track 10.2 -> 34.5 mm, vias 0 -> 1
- net /Counters/~{HSyncClear}: track 0.00 -> 21.5 mm
- net /Counters/Col4: track 7.36 -> 28.6 mm, vias 0 -> 2
- net /Counters/HSyncSet: track 0.00 -> 20.9 mm
- net /Counters/~{HBlankSet}: track 0.00 -> 20.8 mm
- net /Counters/HBlankClear: track 0.00 -> 18.7 mm, vias 0 -> 1
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
Commit message: Row counter logic
Parts:
- moved J13 205.0 mm to (136.5, 98.4)
- moved J14 191.5 mm to (136.5, 79.4)
- moved C26 174.0 mm to (123.8, 144.1), turned to 0 degrees
- moved U26 167.1 mm to (123.8, 137.2), turned to 90 degrees
- moved J9 161.4 mm to (121.9, 128.9), turned to 90 degrees
- moved C27 160.8 mm to (137.8, 144.1), turned to 0 degrees
- moved U27 153.3 mm to (137.8, 137.2), turned to 90 degrees
- moved C28 149.1 mm to (151.8, 144.1), turned to 0 degrees
- moved U28 140.9 mm to (151.8, 137.2), turned to 90 degrees
- moved C21 79.8 mm to (118.1, 118.1), turned to -90 degrees
- moved U21 79.0 mm to (125.7, 118.1), turned to 90 degrees
- moved C25 72.8 mm to (179.4, 106.7)
- moved U25 68.8 mm to (139.1, 91.4), turned to 90 degrees
- moved C19 67.3 mm to (118.1, 109.2), turned to -90 degrees
- moved U19 66.5 mm to (125.7, 109.2), turned to 90 degrees
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Connections:
- U19 pad 10: /Counters/Row6 -> /Counters/Row3
- U19 pad 11: unconnected-(U19-Pad11) -> Net-(U19-Pad11)
- U19 pad 12: GND -> /Counters/HBlankClear
- U19 pad 13: GND -> /Counters/Row0
- U19 pad 2: /Counters/Row0 -> /Counters/Row8
- U19 pad 4: /Counters/HBlankClear -> GND
- U19 pad 5: /Counters/Row0 -> GND
- U19 pad 6: Net-(U19-Pad6) -> unconnected-(U19-Pad6)
- U21 pad 1: Net-(U19-Pad3) -> /Counters/Row0
- U21 pad 12: /Counters/Row8 -> Net-(U19-Pad3)
- U23 pad 1: Net-(U19-Pad6) -> /Counters/Row8
- U23 pad 11: /Counters/Row7 -> Net-(U19-Pad11)
- U23 pad 12: /Counters/Row8 -> Net-(U19-Pad8)
- U23 pad 2: /Counters/~{Row1} -> /Counters/~{Row4}
- U23 pad 3: /Counters/~{Row2} -> /Counters/Row6
- U23 pad 4: /Counters/Row3 -> /Counters/Row7
- U23 pad 5: /Counters/~{Row4} -> /Counters/~{Row2}
- U23 pad 6: Net-(U19-Pad8) -> /Counters/~{Row1}
- U24 pad 1: /Counters/HBlankClear -> /Counters/Row0
- U24 pad 2: /Counters/Row0 -> /Counters/Row1
- U24 pad 3: /Counters/Row1 -> /Counters/HBlankClear
Routing:
- net /Counters/~{VBlankClear}: track 32.8 -> 129.3 mm, vias 0 -> 4
- net /Counters/Row8: track 10.2 -> 82.6 mm, vias 0 -> 3
- net /Counters/Row9: track 8.96 -> 77.4 mm, vias 0 -> 1
- net /Counters/~{HBlankClear}: track 38.5 -> 98.5 mm
- net /Counters/Row2: track 6.83 -> 65.9 mm, vias 0 -> 3
- net /Counters/Row3: track 7.36 -> 66.2 mm, vias 0 -> 3
- net /Counters/Row6: track 6.31 -> 61.2 mm, vias 0 -> 3
- net /Counters/Row5: track 6.83 -> 55.7 mm, vias 0 -> 2
- net /Counters/Row1: track 6.31 -> 55.2 mm, vias 0 -> 3
- net /Counters/Row0: track 5.78 -> 54.0 mm, vias 0 -> 3
- net /Counters/Row4: track 7.36 -> 46.4 mm, vias 0 -> 2
- net Net-(U18-Pad9): track 0.00 -> 23.1 mm
- net /Counters/Row7: track 5.78 -> 27.0 mm, vias 0 -> 1
- net /Counters/VSyncSet: track 0.00 -> 20.9 mm
- net /Counters/VBlankSet: track 0.00 -> 18.9 mm
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Other:
- board text added: "FLIP!"

Commit message: Routing work
Parts:
- J7: footprint footprints:CONN_L77HDE15SD1CH4FVGA_AMP -> Connector_Dsub:DSUB-15-HD_Female_Horizontal_P2.29x1.98mm_EdgePinOffset8.35mm_Housed_MountingHolesOffset10.89mm
- U16, U25: value 74HC109 -> 74AC109
- moved U8 53.4 mm to (113.0, 54.6)
- moved U9 48.0 mm to (97.2, 40.0)
- moved C25 47.9 mm to (134.0, 91.4), turned to -90 degrees
- moved U29 38.7 mm to (150.5, 42.5)
- moved U7 29.6 mm to (81.9, 55.9)
- moved U6 27.5 mm to (95.9, 58.4)
- moved J7 15.9 mm to (230.4, 95.3), turned to 180 degrees
- moved C29 14.7 mm to (98.4, 27.9)
- moved C26 13.3 mm to (110.5, 144.1)
- moved J13 13.3 mm to (123.2, 98.4)
- moved J14 13.3 mm to (123.2, 79.4)
- moved J9 13.3 mm to (108.6, 128.9)
- moved U18 13.3 mm to (112.4, 91.4)
- moved U19 13.3 mm to (112.4, 109.2)
- moved U21 13.3 mm to (112.4, 118.1)
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Connections:
- U19 pad 1: /Counters/HBlankClear -> /Counters/Row0
- U19 pad 12: /Counters/HBlankClear -> /Counters/Row8
- U21 pad 1: /Counters/Row0 -> /Counters/HBlankClear
- U23 pad 1: /Counters/Row8 -> /Counters/~{Row4}
- U23 pad 2: /Counters/~{Row4} -> /Counters/Row6
- U23 pad 3: /Counters/Row6 -> /Counters/Row7
- U23 pad 4: /Counters/Row7 -> /Counters/~{Row2}
- U23 pad 5: /Counters/~{Row2} -> /Counters/~{Row1}
- U23 pad 6: /Counters/~{Row1} -> /Counters/HBlankClear
Routing:
- net /Counters/Row7: track 27.0 -> 126.7 mm, vias 1 -> 3
- net /Counters/PxClock: track 72.1 -> 146.5 mm, vias 0 -> 2
- net /Counters/HBlankClear: track 35.7 -> 101.1 mm, vias 1 -> 3
- net /Counters/Row8: track 82.6 -> 137.2 mm, vias 3 -> 2
- net /Counters/Row6: track 61.2 -> 111.5 mm
- net /Counters/Row5: track 55.7 -> 105.7 mm
- net /Counters/Row3: track 66.2 -> 114.5 mm, vias 3 -> 4
- net /Counters/Row4: track 46.4 -> 94.6 mm
- net /Counters/Row2: track 65.9 -> 110.3 mm
- net /Counters/Col2: track 57.7 -> 101.2 mm
- net /Counters/Col3: track 58.6 -> 101.3 mm
- net /Counters/Col4: track 28.6 -> 70.6 mm
- net +5V: track 80.7 -> 121.5 mm, vias 42 -> 62
- net /Counters/Col5: track 62.0 -> 102.6 mm
- net /Counters/Col6: track 64.2 -> 104.5 mm
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Other:
- board text added: "Buffer A"
- board text added: "Buffer B"
- board text added: "TODO: reorganize pins to simplify routing"

Commit message: Memory routing *screams*
Parts:
- moved C9 60.0 mm to (97.2, 31.5)
- moved C5 54.1 mm to (97.2, 52.5)
- moved C29 49.8 mm to (148.2, 28.2)
- moved U5 49.3 mm to (97.2, 42.0), turned to 180 degrees
- moved C8 37.8 mm to (115.0, 54.7)
- moved C7 33.4 mm to (79.5, 59.4)
- moved U9 19.0 mm to (97.2, 21.0)
- moved U8 9.14 mm to (117.7, 46.8)
- moved U7 6.84 mm to (76.7, 51.4)
- moved U6 4.78 mm to (97.2, 63.0)
Connections:
- U5 pad 1: /Memory/AddrCPU0 -> /Memory/AddrCPU13
- U5 pad 10: /Memory/AddrCPU6 -> /Memory/AddrCPU12
- U5 pad 11: /Memory/AddrB6 -> /Memory/AddrB12
- U5 pad 15: /Memory/AddrCPU8 -> /Memory/AddrCPU6
- U5 pad 16: /Memory/AddrB8 -> /Memory/AddrB6
- U5 pad 17: /Memory/AddrB9 -> /Memory/AddrB5
- U5 pad 18: /Memory/AddrCPU10 -> /Memory/AddrCPU4
- U5 pad 19: /Memory/AddrB10 -> /Memory/AddrB4
- U5 pad 2: /Memory/AddrB0 -> /Memory/AddrB13
- U5 pad 20: /Memory/AddrB11 -> /Memory/AddrB3
- U5 pad 21: /Memory/AddrCPU12 -> /Memory/AddrCPU2
- U5 pad 22: /Memory/AddrB12 -> /Memory/AddrB2
- U5 pad 23: /Memory/AddrB13 -> /Memory/AddrB1
- U5 pad 24: /Memory/AddrCPU14 -> /Memory/AddrCPU0
- U5 pad 25: /Memory/AddrB14 -> /Memory/AddrB0
- U5 pad 3: /Memory/AddrB1 -> /Memory/AddrB8
- U5 pad 33: /Memory/AddrA14 -> /Memory/AddrA0
- U5 pad 34: /Memory/AddrCPU13 -> /Memory/AddrCPU1
- U5 pad 35: /Memory/AddrA13 -> /Memory/AddrA1
- U5 pad 36: /Memory/AddrA12 -> /Memory/AddrA2
- U5 pad 37: /Memory/AddrCPU11 -> /Memory/AddrCPU3
- U5 pad 38: /Memory/AddrA11 -> /Memory/AddrA3
- U5 pad 39: /Memory/AddrA10 -> /Memory/AddrA4
- U5 pad 4: /Memory/AddrCPU2 -> /Memory/AddrCPU9
- U5 pad 40: /Memory/AddrCPU9 -> /Memory/AddrCPU5
- U5 pad 41: /Memory/AddrA9 -> /Memory/AddrA5
- U5 pad 42: /Memory/AddrA8 -> /Memory/AddrA6
- U5 pad 47: /Memory/AddrA6 -> /Memory/AddrA12
- U5 pad 48: /Memory/AddrCPU5 -> /Memory/AddrCPU14
- U5 pad 49: /Memory/AddrA5 -> /Memory/AddrA14
- U5 pad 5: /Memory/AddrB2 -> /Memory/AddrB9
- U5 pad 50: /Memory/AddrA4 -> /Memory/AddrA10
- U5 pad 51: /Memory/AddrCPU3 -> /Memory/AddrCPU11
- U5 pad 52: /Memory/AddrA3 -> /Memory/AddrA11
- U5 pad 53: /Memory/AddrA2 -> /Memory/AddrA9
- U5 pad 54: /Memory/AddrCPU1 -> /Memory/AddrCPU8
- U5 pad 55: /Memory/AddrA1 -> /Memory/AddrA8
- U5 pad 56: /Memory/AddrA0 -> /Memory/AddrA13
- U5 pad 6: /Memory/AddrB3 -> /Memory/AddrB11
- U5 pad 7: /Memory/AddrCPU4 -> /Memory/AddrCPU10
- U5 pad 8: /Memory/AddrB4 -> /Memory/AddrB10
- U5 pad 9: /Memory/AddrB5 -> /Memory/AddrB14
- U6 pad 15: /Counters/Row2 -> /Counters/Row6
- U6 pad 16: /Memory/AddrA8 -> /Memory/AddrA12
- U6 pad 17: /Memory/AddrA9 -> /Memory/AddrA14
- U6 pad 21: /Counters/Row6 -> /Counters/Row3
- U6 pad 22: /Memory/AddrA12 -> /Memory/AddrA9
- U6 pad 23: /Memory/AddrA13 -> /Memory/AddrA8
- U6 pad 24: /Counters/Row8 -> /Counters/Row7
- U6 pad 25: /Memory/AddrA14 -> /Memory/AddrA13
- U6 pad 33: /Memory/AddrB14 -> /Memory/AddrB13
- U6 pad 34: /Counters/Row7 -> /Counters/Row2
- U6 pad 35: /Memory/AddrB13 -> /Memory/AddrB8
- U6 pad 36: /Memory/AddrB12 -> /Memory/AddrB9
- U6 pad 40: /Counters/Row3 -> /Counters/Row8
- U6 pad 41: /Memory/AddrB9 -> /Memory/AddrB14
- U6 pad 42: /Memory/AddrB8 -> /Memory/AddrB12
Routing:
- net /Memory/AddrA6: track 0.00 -> 33.5 mm, vias 0 -> 2
- net /Memory/AddrA4: track 0.00 -> 33.5 mm, vias 0 -> 2
- net /Memory/AddrA2: track 0.00 -> 33.5 mm, vias 0 -> 2
- net /Memory/AddrA12: track 0.00 -> 33.5 mm, vias 0 -> 2
- net /Memory/AddrA0: track 0.00 -> 33.5 mm, vias 0 -> 2
- net /Memory/AddrA5: track 0.00 -> 33.0 mm, vias 0 -> 2
- net /Memory/AddrA3: track 0.00 -> 33.0 mm, vias 0 -> 2
- net /Memory/AddrA14: track 0.00 -> 33.0 mm, vias 0 -> 2
- net /Memory/AddrA1: track 0.00 -> 33.0 mm, vias 0 -> 2
- net /Memory/AddrA7: track 0.00 -> 32.0 mm, vias 0 -> 2
- net /Memory/AddrA9: track 0.00 -> 1.21 mm, vias 0 -> 1
- net /Memory/AddrA8: track 0.00 -> 1.21 mm, vias 0 -> 1
- net /Memory/AddrA13: track 0.00 -> 0.96 mm, vias 0 -> 1
- net /Memory/AddrA11: track 0.00 -> 0.96 mm, vias 0 -> 1
- net /Memory/AddrA10: track 0.00 -> 0.96 mm, vias 0 -> 1
Other:
- board text removed: "TODO: reorganize pins to simplify routing"

Commit message: MOOORE memory routing
Parts:
- moved J2 53.3 mm to (31.8, 15.2)
- moved C8 19.1 mm to (131.7, 64.0)
- moved C7 17.2 mm to (65.4, 49.5), turned to -90 degrees
- moved J4 14.6 mm to (31.8, 38.7)
- moved C6 13.9 mm to (74.4, 16.2)
- moved U8 4.67 mm to (117.7, 51.4)
- moved C9 0.25 mm to (97.2, 31.2)
- moved U9 0.25 mm to (97.2, 20.8)
Connections:
- U9 pad 1: /ConfigReg/DataIn0 -> /ConfigReg/DataIn2
- U9 pad 15: /DAC/PixelOut0 -> /DAC/PixelOut2
- U9 pad 16: /Memory/DataA0 -> /Memory/DataA2
- U9 pad 18: /DAC/PixelOut2 -> /DAC/PixelOut0
- U9 pad 19: /Memory/DataA2 -> /Memory/DataA0
- U9 pad 2: /Memory/DataB0 -> /Memory/DataB2
- U9 pad 39: /Memory/DataB2 -> /Memory/DataB0
- U9 pad 4: /ConfigReg/DataIn2 -> /ConfigReg/DataIn0
- U9 pad 42: /Memory/DataB0 -> /Memory/DataB2
- U9 pad 5: /Memory/DataB2 -> /Memory/DataB0
- U9 pad 53: /Memory/DataA2 -> /Memory/DataA0
- U9 pad 56: /Memory/DataA0 -> /Memory/DataA2
Routing:
- net /Memory/~{BufSel}: track 0.00 -> 76.3 mm, vias 0 -> 3
- net /Memory/AddrB6: track 0.00 -> 52.8 mm, vias 0 -> 2
- net /Memory/AddrB4: track 0.00 -> 52.8 mm, vias 0 -> 2
- net /Memory/AddrB12: track 0.00 -> 52.8 mm, vias 0 -> 2
- net /Memory/AddrB0: track 0.00 -> 52.8 mm, vias 0 -> 2
- net /Memory/AddrB2: track 0.00 -> 52.8 mm, vias 0 -> 2
- net /Memory/BufSel: track 0.00 -> 52.2 mm, vias 0 -> 3
- net /Memory/AddrB5: track 0.00 -> 52.0 mm, vias 0 -> 2
- net /Memory/AddrB3: track 0.00 -> 52.0 mm, vias 0 -> 2
- net /Memory/AddrB14: track 0.00 -> 52.0 mm, vias 0 -> 2
- net /Memory/AddrB1: track 0.00 -> 52.0 mm, vias 0 -> 2
- net /Memory/AddrB7: track 0.00 -> 51.6 mm, vias 0 -> 2
- net /Memory/AddrA10: track 0.96 -> 52.4 mm, vias 1 -> 2
- net /Memory/AddrA11: track 0.96 -> 52.2 mm, vias 1 -> 2
- net /Memory/AddrA8: track 1.21 -> 52.2 mm, vias 1 -> 2
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