File: 6502gpu.kicad_pcb (KiCad board)
At the start: 4 copper layers, 96 parts, among them J1 Conn_01x02, J10 Conn_01x10, J11 Conn_01x03, J12 Conn_01x03, J13 Conn_01x03, J14 Conn_01x03, J15 Conn_01x03, J16 Conn_01x01, J2 Conn_01x08, J3 Conn_01x02, J4 Conn_01x16, J5 Conn_01x02, J6 Conn_01x03, J7 DE15_Receptacle_HighDensity, J8 Conn_01x08, J9 Conn_01x10, U1 74HC86, U10 74AHC30, U11 74AHC30, U12 74AHC30, U13 74AHC30, U14 74LV163, U15 74LV04, U16 74AC109, U17 74LV163, U18 74LV04, U19 74LV08, U2 74HC00, U20 74LV163, U21 74AHC30, U22 74AHC30, U23 74AHC30, U24 74AHC30, U25 74AC109, U26 74LV163, U27 74LV163, U28 74LV163, U29 74HC377, U3 74LV27, U30 74LV32, U31 74LV32, U32 74LV08, U33 74LV08, U4 74HC00, U5 74CBT16390, U6 74CBT16390, U7 AS7C256A-10, U8 AS7C256A-10, U9 74CBT16390, X1 25.175MHz

Commit message: more layout
Parts:
- moved J8 206.4 mm to (116.2, 80.6), turned to -90 degrees
- moved C14 152.5 mm to (217.2, 109.9), turned to 90 degrees
- moved C29 152.0 mm to (298.1, 2.85)
- moved U29 152.0 mm to (300.4, 17.1)
- moved U14 144.2 mm to (210.2, 109.9), turned to 180 degrees
- moved C17 143.0 mm to (217.2, 95.9), turned to 90 degrees
- moved J2 138.1 mm to (96.5, 137.2), turned to 90 degrees
- moved C31 137.0 mm to (92.7, 71.8), turned to -90 degrees
- moved J15 137.0 mm to (87.6, 53.3)
- moved J7 137.0 mm to (103.4, 43.9)
- moved R10 137.0 mm to (114.9, 53.3)
- moved R11 137.0 mm to (104.8, 53.3)
- moved R2 137.0 mm to (117.5, 53.3)
- moved R3 137.0 mm to (112.4, 53.3)
- moved R5 137.0 mm to (107.3, 53.3)
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Routing:
- net /Memory/AddrCPU8: track 0.00 -> 60.2 mm, vias 0 -> 1
- net /Memory/AddrCPU9: track 1.04 -> 56.7 mm
- net /Memory/AddrCPU10: track 1.04 -> 56.2 mm
- net /Memory/AddrCPU12: track 1.54 -> 56.4 mm
- net /Memory/AddrCPU11: track 0.00 -> 52.8 mm, vias 0 -> 1
- net /Memory/AddrCPU6: track 0.00 -> 51.2 mm, vias 0 -> 1
- net /Memory/AddrCPU4: track 1.54 -> 49.3 mm
- net /Memory/AddrCPU2: track 1.04 -> 47.4 mm
- net /Memory/AddrCPU7: track 1.04 -> 45.4 mm
- net /Memory/AddrCPU0: track 1.54 -> 45.8 mm
- net /Memory/AddrCPU5: track 1.04 -> 42.7 mm
- net /Memory/AddrCPU3: track 1.04 -> 40.8 mm
- net /DAC/PixelOut0: track 0.00 -> 39.3 mm, vias 0 -> 1
- net /Memory/AddrCPU1: track 1.04 -> 38.9 mm
- net /DAC/PixelOut2: track 0.00 -> 34.0 mm, vias 0 -> 2
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Other:
- board outline added: 146.7 x 110.5 mm
- board text added: "VGA Specs: 160x120 (scaled to 640x480) 256 Colors (332 RGB)"

Commit message: layout continues...
Parts:
- added J17: Barrel_Jack, Connector_BarrelJack:BarrelJack_CUI_PJ-102AH_Horizontal, F.Cu at (214.3, 122.6)
- added U34: LM7805, Package_TO_SOT_THT:TO-220-3_Vertical, F.Cu at (209.6, 122.6)
- moved C1 305.5 mm to (7.28, 92.4)
- moved C3 305.5 mm to (26.3, 89.9)
- moved U2 305.5 mm to (17.1, 102.2)
- moved U3 305.5 mm to (25.6, 102.2)
- moved U4 305.5 mm to (68.0, 107.0)
- moved C2 305.5 mm to (15.5, 90.5)
- moved C4 305.5 mm to (68.3, 114.3)
- moved U1 305.5 mm to (8.66, 102.2)
- moved C29 241.5 mm to (90.2, 125.7), turned to -90 degrees
- moved U29 228.2 mm to (99.7, 125.7), turned to 90 degrees
- moved J3 148.5 mm to (177.8, 137.2), turned to 90 degrees
- moved J5 142.9 mm to (170.2, 137.2), turned to 90 degrees
- moved C35 141.5 mm to (179.1, 130.2), turned to 0 degrees
- moved J1 138.2 mm to (162.6, 137.2), turned to 90 degrees
- moved C34 50.0 mm to (192.4, 90.8)
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Connections:
- net /Memory/BufSel renamed /ConfigReg/BufSel
- U29 pad 14: /ConfigReg/DataIn5 -> GND
- U29 pad 17: /ConfigReg/DataIn6 -> GND
- U29 pad 18: /ConfigReg/DataIn7 -> GND
Routing:
- net /ConfigReg/DataIn3: track 0.00 -> 61.1 mm, vias 0 -> 1
- net /ConfigReg/DataIn1: track 0.00 -> 59.6 mm, vias 0 -> 1
- net /ConfigReg/DataIn4: track 0.00 -> 58.8 mm, vias 0 -> 1
- net /ConfigReg/DataIn7: track 0.00 -> 58.5 mm, vias 0 -> 1
- net /ConfigReg/DataIn5: track 0.00 -> 56.1 mm, vias 0 -> 1
- net /Counters/Row8: track 137.2 -> 82.8 mm
- net /Counters/Row7: track 126.7 -> 74.3 mm
- net /Counters/Row6: track 111.5 -> 59.6 mm
- net /Counters/PxClock: track 149.5 -> 200.4 mm, vias 2 -> 0
- net /Counters/Row5: track 105.7 -> 55.7 mm
- net /ConfigReg/DataIn0: track 0.00 -> 48.2 mm, vias 0 -> 1
- net /Counters/Row4: track 94.6 -> 46.4 mm
- net /ConfigReg/DataIn2: track 0.00 -> 47.1 mm, vias 0 -> 1
- net /Counters/Row3: track 114.5 -> 68.6 mm
- net /Counters/Row2: track 110.3 -> 66.0 mm
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Other:
- board text added: "Config Register"
- board text added: "Control"
- board text added: "HBlank / HSync"
- board text added: "Power"
- board text added: "VBlank / VSync"
- board text added: "~{FbSel} pulled low when CPU is accessing this board's address space"
- board text added: "~{NMI} pulled low at start of vertical blank if NmiEnable set"
- board text removed: "Counters"

Commit message: finalize board layout at 140x110mm
Parts:
- added REF**: MountingHole_3.2mm_M3, MountingHole:MountingHole_3.2mm_M3, F.Cu at (220.5, 137.8)
- added REF**: MountingHole_3.2mm_M3, MountingHole:MountingHole_3.2mm_M3, F.Cu at (87.5, 137.8)
- added REF**: MountingHole_3.2mm_M3, MountingHole:MountingHole_3.2mm_M3, F.Cu at (87.5, 34.8)
- added REF**: MountingHole_3.2mm_M3, MountingHole:MountingHole_3.2mm_M3, F.Cu at (220.5, 34.8)
- moved C1 165.3 mm to (168.9, 127.0), turned to -90 degrees
- moved U1 154.6 mm to (161.3, 127.0), turned to 90 degrees
- moved C2 142.9 mm to (153.7, 127.0), turned to -90 degrees
- moved U2 131.3 mm to (146.1, 127.0), turned to 90 degrees
- moved J6 116.5 mm to (143.5, 116.8), turned to 90 degrees
- moved U3 68.3 mm to (90.8, 81.9)
- moved C3 64.5 mm to (90.8, 89.5)
- moved U4 55.4 mm to (122.6, 116.8)
- moved J17 5.99 mm to (209.3, 125.7)
- moved U34 5.99 mm to (204.5, 125.7)
- moved C4 3.15 mm to (65.4, 115.6)
Connections:
- U3 pad 10: /~{RegSel} -> /~{FbSelected}
- U3 pad 3: /~{FbSelected} -> /~{Phi2}
- U3 pad 4: /~{Phi2} -> /R~{W}
- U3 pad 5: /R~{W} -> /~{FbSelected}
- U3 pad 9: /~{FbSelected} -> /~{RegSel}
Routing:
- net /VBlank: track 7.00 -> 136.9 mm, vias 0 -> 2
- net /HBlank: track 7.80 -> 126.5 mm, vias 0 -> 3
- net /~{HSync}: track 12.5 -> 97.2 mm
- net /Counters/Row4: track 46.4 -> 103.7 mm, vias 2 -> 3
- net /Counters/Row6: track 59.6 -> 111.6 mm, vias 3 -> 4
- net /~{VSync}: track 12.5 -> 61.9 mm, vias 0 -> 1
- net /Counters/Row7: track 74.3 -> 122.2 mm, vias 3 -> 4
- net /ConfigReg/BlankBlack: track 0.00 -> 46.6 mm
- net /Counters/Row8: track 82.8 -> 122.8 mm, vias 2 -> 3
- net /Memory/AddrCPU13: track 21.0 -> 60.8 mm
- net /Counters/Row5: track 55.7 -> 93.8 mm, vias 2 -> 3
- net /Counters/Row3: track 68.6 -> 105.8 mm, vias 4 -> 5
- net /AddrPhys14: track 0.00 -> 33.8 mm
- net /~{FbSelected}: track 0.00 -> 32.7 mm, vias 0 -> 1
- net /AddrPhys15: track 0.00 -> 32.2 mm
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Other:
- board size 146.7 x 110.5 mm -> 140 x 110 mm
- board text added: "6502 VGA Adapter Gary Bailey"
- board text removed: "VRAM"

Commit message: almost done wiring...
Parts:
- removed REF** (x4): MountingHole_3.2mm_M3, MountingHole:MountingHole_3.2mm_M3
- added H1: MountingHole, MountingHole:MountingHole_3.2mm_M3, F.Cu at (87.5, 34.8)
- added H2: MountingHole, MountingHole:MountingHole_3.2mm_M3, F.Cu at (220.5, 34.8)
- added H3: MountingHole, MountingHole:MountingHole_3.2mm_M3, F.Cu at (87.5, 137.8)
- added H4: MountingHole, MountingHole:MountingHole_3.2mm_M3, F.Cu at (220.5, 137.8)
Connections:
- net /~{FbSelected} renamed /~{FbSel}
- U2 pad 1: /VBlank -> /Memory/AddrCPU5
- U2 pad 11: /~{RegSel} -> /~{NMI}
- U2 pad 12: /Memory/AddrCPU5 -> /VBlank
- U2 pad 13: /Memory/AddrCPU7 -> /ConfigReg/NmiEnable
- U2 pad 2: /ConfigReg/NmiEnable -> /Memory/AddrCPU7
- U2 pad 3: /~{NMI} -> /~{RegSel}
Routing:
- net /ConfigReg/BlankWhite: track 24.9 -> 110.9 mm, vias 2 -> 5
- net GND: track 72.2 -> 108.6 mm, vias 29 -> 40
- net Net-(U1-Pad3): track 0.00 -> 20.8 mm
- net /DAC/PixelOut7: track 28.6 -> 45.1 mm
- net /Memory/AddrCPU5: track 42.7 -> 56.0 mm
- net /DAC/PixelOut4: track 29.2 -> 42.2 mm
- net /ConfigReg/DataIn4: track 58.8 -> 46.3 mm, vias 1 -> 2
- net +5V: track 156.3 -> 167.4 mm, vias 80 -> 83
- net /Memory/AddrCPU7: track 45.4 -> 55.7 mm
- net /DAC/PixelOut6: track 33.9 -> 42.7 mm
- net /DAC/PixelOut5: track 23.0 -> 30.5 mm
- net /~{NMI}: track 29.0 -> 34.3 mm
- net /Counters/Row9: track 77.4 -> 73.3 mm
- net /~{RegSel}: track 0.00 -> 0.73 mm
- net /DAC/PixelOut0: track 39.3 -> 38.7 mm
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