File: memory.kicad_sch (KiCad schematic)
At the start: 7 parts, among them U1 62256, U3 74CBT16390, U4 74CBT16390, U5 74CBT3390, U6 74CBT3390, U7 74HC00

Commit message: cleanup
Connections:
- removed net A0: U1.10 (A0), U1.10 (A0), U3.1 (A1), U3.2 (2B1), U3.56 (1B1), U4.1 (A1), U4.2 (2B1), U4.56 (1B1)
- removed net A1: U1.9 (A1), U1.9 (A1), U3.3 (2B2), U3.54 (A2), U3.55 (1B2), U4.3 (2B2), U4.54 (A2), U4.55 (1B2)
- removed net A10: U1.21 (A10), U1.21 (A10), U3.18 (A11), U3.19 (2B11), U3.39 (1B11), U4.18 (A11), U4.19 (2B11), U4.39 (1B11)
- removed net A11: U1.23 (A11), U1.23 (A11), U3.20 (2B12), U3.37 (A12), U3.38 (1B12), U4.20 (2B12), U4.37 (A12), U4.38 (1B12)
- removed net A12: U1.2 (A12), U1.2 (A12), U3.21 (A13), U3.22 (2B13), U3.36 (1B13), U4.21 (A13), U4.22 (2B13), U4.36 (1B13)
- removed net A13: U1.26 (A13), U1.26 (A13), U3.23 (2B14), U3.34 (A14), U3.35 (1B14), U4.23 (2B14), U4.34 (A14), U4.35 (1B14)
- removed net A14: U1.1 (A14), U1.1 (A14), U3.24 (A15), U3.25 (2B15), U3.33 (1B15), U4.24 (A15), U4.25 (2B15), U4.33 (1B15)
- removed net A2: U1.8 (A2), U1.8 (A2), U3.4 (A3), U3.5 (2B3), U3.53 (1B3), U4.4 (A3), U4.5 (2B3), U4.53 (1B3)
- removed net A3: U1.7 (A3), U1.7 (A3), U3.51 (A4), U3.52 (1B4), U3.6 (2B4), U4.51 (A4), U4.52 (1B4), U4.6 (2B4)
- removed net A4: U1.6 (A4), U1.6 (A4), U3.50 (1B5), U3.7 (A5), U3.8 (2B5), U4.50 (1B5), U4.7 (A5), U4.8 (2B5)
- removed net A5: U1.5 (A5), U1.5 (A5), U3.48 (A6), U3.49 (1B6), U3.9 (2B6), U4.48 (A6), U4.49 (1B6), U4.9 (2B6)
- removed net A6: U1.4 (A6), U1.4 (A6), U3.10 (A7), U3.11 (2B7), U3.47 (1B7), U4.10 (A7), U4.11 (2B7), U4.47 (1B7)
- removed net A7: U1.3 (A7), U1.3 (A7), U3.12 (2B8), U3.45 (A8), U3.46 (1B8), U4.12 (2B8), U4.45 (A8), U4.46 (1B8)
- removed net A8: U1.25 (A8), U1.25 (A8), U3.15 (A9), U3.16 (2B9), U3.42 (1B9), U4.15 (A9), U4.16 (2B9), U4.42 (1B9)
- removed net A9: U1.24 (A9), U1.24 (A9), U3.17 (2B10), U3.40 (A10), U3.41 (1B10), U4.17 (2B10), U4.40 (A10), U4.41 (1B10)
- removed net D0: U1.11 (Q0), U1.11 (Q0), U5.1 (1B1), U5.2 (2B1), U5.3 (A1), U6.1 (1B1), U6.2 (2B1), U6.3 (A1)
- removed net D1: U1.12 (Q1), U1.12 (Q1), U5.4 (1B2), U5.5 (2B2), U5.6 (A2), U6.4 (1B2), U6.5 (2B2), U6.6 (A2)
- removed net D2: U1.13 (Q2), U1.13 (Q2), U5.7 (1B3), U5.8 (2B3), U5.9 (A3), U6.7 (1B3), U6.8 (2B3), U6.9 (A3)
- removed net D3: U1.15 (Q3), U1.15 (Q3), U5.10 (1B4), U5.11 (2B4), U5.12 (A4), U6.10 (1B4), U6.11 (2B4), U6.12 (A4)
- removed net D4: U1.16 (Q4), U1.16 (Q4), U5.16 (A5), U5.17 (2B5), U5.18 (1B5), U6.16 (A5), U6.17 (2B5), U6.18 (1B5)
- removed net D5: U1.17 (Q5), U1.17 (Q5), U5.19 (A6), U5.20 (2B6), U5.21 (1B6), U6.19 (A6), U6.20 (2B6), U6.21 (1B6)
- removed net D6: U1.18 (Q6), U1.18 (Q6), U5.22 (A7), U5.23 (2B7), U5.24 (1B7), U6.22 (A7), U6.23 (2B7), U6.24 (1B7)
- removed net D7: U1.19 (Q7), U1.19 (Q7), U5.25 (A8), U5.26 (2B8), U5.27 (1B8), U6.25 (A8), U6.26 (2B8), U6.27 (1B8)
- new net AddrA0: U1.10 (A0), U3.56 (1B1), U4.2 (2B1)
- new net AddrA1: U1.9 (A1), U3.55 (1B2), U4.3 (2B2)
- new net AddrA10: U1.21 (A10), U3.39 (1B11), U4.19 (2B11)
- new net AddrA11: U1.23 (A11), U3.38 (1B12), U4.20 (2B12)
- new net AddrA12: U1.2 (A12), U3.36 (1B13), U4.22 (2B13)
- new net AddrA13: U1.26 (A13), U3.35 (1B14), U4.23 (2B14)
- new net AddrA14: U1.1 (A14), U3.33 (1B15), U4.25 (2B15)
- new net AddrA2: U1.8 (A2), U3.53 (1B3), U4.5 (2B3)
- new net AddrA3: U1.7 (A3), U3.52 (1B4), U4.6 (2B4)
- new net AddrA4: U1.6 (A4), U3.50 (1B5), U4.8 (2B5)
- new net AddrA5: U1.5 (A5), U3.49 (1B6), U4.9 (2B6)
- new net AddrA6: U1.4 (A6), U3.47 (1B7), U4.11 (2B7)
- new net AddrA7: U1.3 (A7), U3.46 (1B8), U4.12 (2B8)
- new net AddrA8: U1.25 (A8), U3.42 (1B9), U4.16 (2B9)
- new net AddrA9: U1.24 (A9), U3.41 (1B10), U4.17 (2B10)
- new net AddrB0: U1.10 (A0), U3.2 (2B1), U4.56 (1B1)
- new net AddrB1: U1.9 (A1), U3.3 (2B2), U4.55 (1B2)
- new net AddrB10: U1.21 (A10), U3.19 (2B11), U4.39 (1B11)
- new net AddrB11: U1.23 (A11), U3.20 (2B12), U4.38 (1B12)
- new net AddrB12: U1.2 (A12), U3.22 (2B13), U4.36 (1B13)
- new net AddrB13: U1.26 (A13), U3.23 (2B14), U4.35 (1B14)
- new net AddrB14: U1.1 (A14), U3.25 (2B15), U4.33 (1B15)
- new net AddrB2: U1.8 (A2), U3.5 (2B3), U4.53 (1B3)
- new net AddrB3: U1.7 (A3), U3.6 (2B4), U4.52 (1B4)
- new net AddrB4: U1.6 (A4), U3.8 (2B5), U4.50 (1B5)
- new net AddrB5: U1.5 (A5), U3.9 (2B6), U4.49 (1B6)
- new net AddrB6: U1.4 (A6), U3.11 (2B7), U4.47 (1B7)
- new net AddrB7: U1.3 (A7), U3.12 (2B8), U4.46 (1B8)
- new net AddrB8: U1.25 (A8), U3.16 (2B9), U4.42 (1B9)
- new net AddrB9: U1.24 (A9), U3.17 (2B10), U4.41 (1B10)
- new net AddrCPU0: U3.1 (A1)
- new net AddrCPU1: U3.54 (A2)
- new net AddrCPU10: U3.18 (A11)
- new net AddrCPU11: U3.37 (A12)
- new net AddrCPU12: U3.21 (A13)
- new net AddrCPU13: U3.34 (A14)
- new net AddrCPU14: U3.24 (A15)
- new net AddrCPU2: U3.4 (A3)
- new net AddrCPU3: U3.51 (A4)
- new net AddrCPU4: U3.7 (A5)
- new net AddrCPU5: U3.48 (A6)
- new net AddrCPU6: U3.10 (A7)
- new net AddrCPU7: U3.45 (A8)
- new net AddrCPU8: U3.15 (A9)
- new net AddrCPU9: U3.40 (A10)
- new net AddrGPU0: U4.1 (A1)
- new net AddrGPU1: U4.54 (A2)
- new net AddrGPU10: U4.18 (A11)
- new net AddrGPU11: U4.37 (A12)
- new net AddrGPU12: U4.21 (A13)
- new net AddrGPU13: U4.34 (A14)
- new net AddrGPU14: U4.24 (A15)
- new net AddrGPU2: U4.4 (A3)
- new net AddrGPU3: U4.51 (A4)
- new net AddrGPU4: U4.7 (A5)
- new net AddrGPU5: U4.48 (A6)
- new net AddrGPU6: U4.10 (A7)
- new net AddrGPU7: U4.45 (A8)
- new net AddrGPU8: U4.15 (A9)
- new net AddrGPU9: U4.40 (A10)
- new net DataA0: U1.11 (Q0), U5.1 (1B1), U6.2 (2B1)
- new net DataA1: U1.12 (Q1), U5.4 (1B2), U6.5 (2B2)
- new net DataA2: U1.13 (Q2), U5.7 (1B3), U6.8 (2B3)
- new net DataA3: U1.15 (Q3), U5.10 (1B4), U6.11 (2B4)
- new net DataA4: U1.16 (Q4), U5.18 (1B5), U6.17 (2B5)
- new net DataA5: U1.17 (Q5), U5.21 (1B6), U6.20 (2B6)
- new net DataA6: U1.18 (Q6), U5.24 (1B7), U6.23 (2B7)
- new net DataA7: U1.19 (Q7), U5.27 (1B8), U6.26 (2B8)
- new net DataB0: U1.11 (Q0), U5.2 (2B1), U6.1 (1B1)
- new net DataB1: U1.12 (Q1), U5.5 (2B2), U6.4 (1B2)
- new net DataB2: U1.13 (Q2), U5.8 (2B3), U6.7 (1B3)
- new net DataB3: U1.15 (Q3), U5.11 (2B4), U6.10 (1B4)
- new net DataB4: U1.16 (Q4), U5.17 (2B5), U6.18 (1B5)
- new net DataB5: U1.17 (Q5), U5.20 (2B6), U6.21 (1B6)
- new net DataB6: U1.18 (Q6), U5.23 (2B7), U6.24 (1B7)
- new net DataB7: U1.19 (Q7), U5.26 (2B8), U6.27 (1B8)
- new net DataCPU0: U5.3 (A1)
- new net DataCPU1: U5.6 (A2)
- new net DataCPU2: U5.9 (A3)
- new net DataCPU3: U5.12 (A4)
- new net DataCPU4: U5.16 (A5)
- new net DataCPU5: U5.19 (A6)
- new net DataCPU6: U5.22 (A7)
- new net DataCPU7: U5.25 (A8)
- new net DataGPU0: U6.3 (A1)
- new net DataGPU1: U6.6 (A2)
- new net DataGPU2: U6.9 (A3)
- new net DataGPU3: U6.12 (A4)
- new net DataGPU4: U6.16 (A5)
- new net DataGPU5: U6.19 (A6)
- new net DataGPU6: U6.22 (A7)
- new net DataGPU7: U6.25 (A8)
Other:
- moved on the sheet: U3, U4, U7A, U7B, U7C, U7D, U7E

Commit message: remove 3390, cleanup
Parts:
- removed U5, U6: 74CBT3390, symbol custom:74CBT3390
- added U33: 74CBT16390, symbol custom:74CBT16390
Connections:
- net +5V: now also U33.14 (V_{CC}), U33.43 (V_{CC})
- net BufSel: now also U33.30 (~{OE1})
- net DataA0: now also U33.16 (2B9), U33.56 (1B1)
- net DataA1: now also U33.17 (2B10), U33.55 (1B2)
- net DataA2: now also U33.19 (2B11), U33.53 (1B3)
- net DataA3: now also U33.20 (2B12), U33.52 (1B4)
- net DataA4: now also U33.22 (2B13), U33.50 (1B5)
- net DataA5: now also U33.23 (2B14), U33.49 (1B6)
- net DataA6: now also U33.25 (2B15), U33.47 (1B7)
- net DataA7: now also U33.26 (2B16), U33.46 (1B8)
- net DataB0: now also U33.2 (2B1), U33.42 (1B9)
- net DataB1: now also U33.3 (2B2), U33.41 (1B10)
- net DataB2: now also U33.39 (1B11), U33.5 (2B3)
- net DataB3: now also U33.38 (1B12), U33.6 (2B4)
- net DataB4: now also U33.36 (1B13), U33.8 (2B5)
- net DataB5: now also U33.35 (1B14), U33.9 (2B6)
- net DataB6: now also U33.11 (2B7), U33.33 (1B15)
- net DataB7: now also U33.12 (2B8), U33.32 (1B16)
- net DataCPU0: now also U33.1 (A1)
- net DataCPU1: now also U33.54 (A2)
- net DataCPU2: now also U33.4 (A3)
- net DataCPU3: now also U33.51 (A4)
- net DataCPU4: now also U33.7 (A5)
- net DataCPU5: now also U33.48 (A6)
- net DataCPU6: now also U33.10 (A7)
- net DataCPU7: now also U33.45 (A8)
- net GND: now also U33.13 (GND), U33.44 (GND)
- net AddrGPU0 renamed Col2
- net AddrGPU1 renamed Col3
- net AddrGPU10 renamed Row4
- net AddrGPU11 renamed Row5
- net AddrGPU12 renamed Row6
- net AddrGPU13 renamed Row7
- net AddrGPU14 renamed Row8
- net AddrGPU2 renamed Col4
- net AddrGPU3 renamed Col5
- net AddrGPU4 renamed Col6
- net AddrGPU5 renamed Col7
- net AddrGPU6 renamed Col8
- net AddrGPU7 renamed Col9
- net AddrGPU8 renamed Row2
- net AddrGPU9 renamed Row3
- net ~{BufSelY} renamed ~{BufSel}
- net ~{BufSel}: now also U33.29 (~{OE2})
- new net PixelOut0: U33.15 (A9)
- new net PixelOut1: U33.40 (A10)
- new net PixelOut2: U33.18 (A11)
- new net PixelOut3: U33.37 (A12)
- new net PixelOut4: U33.21 (A13)
- new net PixelOut5: U33.34 (A14)
- new net PixelOut6: U33.24 (A15)
- new net PixelOut7: U33.31 (A16)
Other:
- note added: "If BufSel is LOW: - CPU connects to Buffer A - GPU connects to Buffer B - Buffer B outputs If BufSel is HIGH: - CPU connects to Buffer B - GPU connects to Buffer A - Buffer A outputs"
- note removed: "~{BufSelX} and ~{BufSelY} form a 1-hot pair If ~{BufSelX} is LOW, state X is active If ~{BufSelY} is LOW, state Y is active State X: CPU connects to Buffer A, GPU connects to Buffer B State Y: CPU connects to Buffer B, GPU connects to Buffer A BufSel LOW selects state X, HIGH selects state Y"
- moved on the sheet: U1

Commit message: work on main page layout
Connections:
- net DataCPU0 renamed DataIn0
- net DataCPU1 renamed DataIn1
- net DataCPU2 renamed DataIn2
- net DataCPU3 renamed DataIn3
- net DataCPU4 renamed DataIn4
- net DataCPU5 renamed DataIn5
- net DataCPU6 renamed DataIn6
- net DataCPU7 renamed DataIn7
- net WriteCPU renamed WriteMem
Changed lines of the file:
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@@
     (effects (font (size 1.27 1.27)) (justify right bottom))
   )
-  (label "DataCPU7" (at 241.3 68.58 180) (fields_autoplaced)
+  (label "DataIn7" (at 241.3 68.58 180) (fields_autoplaced)
     (effects (font (size 1.27 1.27)) (justify right bottom))
   )
@@
     (effects (font (size 1.27 1.27)) (justify right bottom))
   )
-  (label "DataCPU6" (at 241.3 66.04 180) (fields_autoplaced)
+  (label "DataIn6" (at 241.3 66.04 180) (fields_autoplaced)
     (effects (font (size 1.27 1.27)) (justify right bottom))
   )
@@
     (effects (font (size 1.27 1.27)) (justify right bottom))
   )
-  (label "DataCPU1" (at 241.3 53.34 180) (fields_autoplaced)
+  (label "DataIn1" (at 241.3 53.34 180) (fields_autoplaced)
     (effects (font (size 1.27 1.27)) (justify right bottom))
   )
@@
     (effects (font (size 1.27 1.27)) (justify left bottom))
   )
-  (label "DataCPU5" (at 241.3 63.5 180) (fields_autoplaced)
+  (label "DataIn5" (at 241.3 63.5 180) (fields_autoplaced)
     (effects (font (size 1.27 1.27)) (justify right bottom))
   )
@@
     (effects (font (size 1.27 1.27)) (justify left bottom))
   )
-  (label "DataCPU2" (at 241.3 55.88 180) (fields_autoplaced)
+  (label "DataIn2" (at 241.3 55.88 180) (fields_autoplaced)
     (effects (font (size 1.27 1.27)) (justify right bottom))
   )
@@
     (effects (font (size 1.27 1.27)) (justify left bottom))
   )
-  (label "DataCPU3" (at 241.3 58.42 180) (fields_autoplaced)
+  (label "DataIn3" (at 241.3 58.42 180) (fields_autoplaced)
     (effects (font (size 1.27 1.27)) (justify right bottom))
   )
@@
     (effects (font (size 1.27 1.27)) (justify right bottom))
   )
-  (label "DataCPU4" (at 241.3 60.96 180) (fields_autoplaced)
+  (label "DataIn4" (at 241.3 60.96 180) (fields_autoplaced)
     (effects (font (size 1.27 1.27)) (justify right bottom))
   )
@@
     (effects (font (size 1.27 1.27)) (justify left bottom))
   )
-  (label "DataCPU0" (at 241.3 50.8 180) (fields_autoplaced)
+  (label "DataIn0" (at 241.3 50.8 180) (fields_autoplaced)
     (effects (font (size 1.27 1.27)) (justify right bottom))
   )
@@
     (effects (font (size 1.27 1.27)) (justify right))
   )
-  (hierarchical_label "DataCPU[0..7]" (shape input) (at 243.84 71.12 0) (fields_autoplaced)
+  (hierarchical_label "DataIn[0..7]" (shape input) (at 243.84 71.12 0) (fields_autoplaced)
     (effects (font (size 1.27 1.27)) (justify left))
   )
@@
     (effects (font (size 1.27 1.27)) (justify right))
   )
-  (hierarchical_label "WriteCPU" (shape input) (at 38.1 96.52 180) (fields_autoplaced)
+  (hierarchical_label "WriteMem" (shape input) (at 38.1 96.52 180) (fields_autoplaced)
     (effects (font (size 1.27 1.27)) (justify right))
   )
-  (hierarchical_label "Row[2..9]" (shape input) (at 69.85 152.4 180) (fields_autoplaced)
+  (hierarchical_label "Row[0..9]" (shape input) (at 69.85 152.4 180) (fields_autoplaced)
     (effects (font (size 1.27 1.27)) (justify right))
   )

Commit message: misc fixes, start on pcb
Parts:
- removed unit 5 of U7
- added C1 (x5): 0.1u, Capacitor_SMD:C_1206_3216Metric_Pad1.33x1.80mm_HandSolder, symbol Device:C
- U1: value 62256 -> AS7C256A-10; footprint Package_DIP:DIP-28_W15.24mm -> Package_SO:TSOP-I-28_11.8x8mm_P0.55mm
- U4: renamed from U7; footprint (none) -> Package_SO:SOIC-14_3.9x8.7mm_P1.27mm
- U5: renamed from U3; footprint (none) -> Package_SO:TSSOP-56_6.1x14mm_P0.5mm
- U6: renamed from U4; footprint (none) -> Package_SO:TSSOP-56_6.1x14mm_P0.5mm
- U9: renamed from U33; footprint (none) -> Package_SO:TSSOP-56_6.1x14mm_P0.5mm
Connections:
- net +5V: now also C1.1, C1.1, C1.1, C1.1, C1.1
- net GND: now also C1.2, C1.2, C1.2, C1.2, C1.2

Commit message: Memory routing *screams*
Connections:
- net AddrA0: now also U5.33 (1B15); no longer U5.56 (1B1)
- net AddrA1: now also U5.35 (1B14); no longer U5.55 (1B2)
- net AddrA10: now also U5.50 (1B5); no longer U5.39 (1B11)
- net AddrA11: now also U5.52 (1B4); no longer U5.38 (1B12)
- net AddrA12: now also U5.47 (1B7), U6.16 (2B9); no longer U5.36 (1B13), U6.22 (2B13)
- net AddrA13: now also U5.56 (1B1), U6.25 (2B15); no longer U5.35 (1B14), U6.23 (2B14)
- net AddrA14: now also U5.49 (1B6), U6.17 (2B10); no longer U5.33 (1B15), U6.25 (2B15)
- net AddrA2: now also U5.36 (1B13); no longer U5.53 (1B3)
- net AddrA3: now also U5.38 (1B12); no longer U5.52 (1B4)
- net AddrA4: now also U5.39 (1B11); no longer U5.50 (1B5)
- net AddrA5: now also U5.41 (1B10); no longer U5.49 (1B6)
- net AddrA6: now also U5.42 (1B9); no longer U5.47 (1B7)
- net AddrA8: now also U5.55 (1B2), U6.23 (2B14); no longer U5.42 (1B9), U6.16 (2B9)
- net AddrA9: now also U5.53 (1B3), U6.22 (2B13); no longer U5.41 (1B10), U6.17 (2B10)
- net AddrB0: now also U5.25 (2B15); no longer U5.2 (2B1)
- net AddrB1: now also U5.23 (2B14); no longer U5.3 (2B2)
- net AddrB10: now also U5.8 (2B5); no longer U5.19 (2B11)
- net AddrB11: now also U5.6 (2B4); no longer U5.20 (2B12)
- net AddrB12: now also U5.11 (2B7), U6.42 (1B9); no longer U5.22 (2B13), U6.36 (1B13)
- net AddrB13: now also U5.2 (2B1), U6.33 (1B15); no longer U5.23 (2B14), U6.35 (1B14)
- net AddrB14: now also U5.9 (2B6), U6.41 (1B10); no longer U5.25 (2B15), U6.33 (1B15)
- net AddrB2: now also U5.22 (2B13); no longer U5.5 (2B3)
- net AddrB3: now also U5.20 (2B12); no longer U5.6 (2B4)
- net AddrB4: now also U5.19 (2B11); no longer U5.8 (2B5)
- net AddrB5: now also U5.17 (2B10); no longer U5.9 (2B6)
- net AddrB6: now also U5.16 (2B9); no longer U5.11 (2B7)
- net AddrB8: now also U5.3 (2B2), U6.35 (1B14); no longer U5.16 (2B9), U6.42 (1B9)
- net AddrB9: now also U5.5 (2B3), U6.36 (1B13); no longer U5.17 (2B10), U6.41 (1B10)
- net AddrCPU0: now also U5.24 (A15); no longer U5.1 (A1)
- net AddrCPU1: now also U5.34 (A14); no longer U5.54 (A2)
- net AddrCPU10: now also U5.7 (A5); no longer U5.18 (A11)
- net AddrCPU11: now also U5.51 (A4); no longer U5.37 (A12)
- net AddrCPU12: now also U5.10 (A7); no longer U5.21 (A13)
- net AddrCPU13: now also U5.1 (A1); no longer U5.34 (A14)
- net AddrCPU14: now also U5.48 (A6); no longer U5.24 (A15)
- net AddrCPU2: now also U5.21 (A13); no longer U5.4 (A3)
- net AddrCPU3: now also U5.37 (A12); no longer U5.51 (A4)
- net AddrCPU4: now also U5.18 (A11); no longer U5.7 (A5)
- net AddrCPU5: now also U5.40 (A10); no longer U5.48 (A6)
- net AddrCPU6: now also U5.15 (A9); no longer U5.10 (A7)
- net AddrCPU8: now also U5.54 (A2); no longer U5.15 (A9)
- net AddrCPU9: now also U5.4 (A3); no longer U5.40 (A10)
- net Row2: now also U6.34 (A14); no longer U6.15 (A9)
- net Row3: now also U6.21 (A13); no longer U6.40 (A10)
- net Row6: now also U6.15 (A9); no longer U6.21 (A13)
- net Row7: now also U6.24 (A15); no longer U6.34 (A14)
- net Row8: now also U6.40 (A10); no longer U6.24 (A15)

Commit message: MOOORE memory routing
Connections:
- net DataA0: now also U9.19 (2B11), U9.53 (1B3); no longer U9.16 (2B9), U9.56 (1B1)
- net DataA2: now also U9.16 (2B9), U9.56 (1B1); no longer U9.19 (2B11), U9.53 (1B3)
- net DataB0: now also U9.39 (1B11), U9.5 (2B3); no longer U9.2 (2B1), U9.42 (1B9)
- net DataB2: now also U9.2 (2B1), U9.42 (1B9); no longer U9.39 (1B11), U9.5 (2B3)
- net DataIn0: now also U9.4 (A3); no longer U9.1 (A1)
- net DataIn2: now also U9.1 (A1); no longer U9.4 (A3)
- net PixelOut0: now also U9.18 (A11); no longer U9.15 (A9)
- net PixelOut2: now also U9.15 (A9); no longer U9.18 (A11)
Changed lines of the file:
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@@
     (effects (font (size 1.27 1.27)) (justify left bottom))
   )
-  (label "DataB0" (at 193.04 71.12 0) (fields_autoplaced)
+  (label "DataB0" (at 193.04 76.2 0) (fields_autoplaced)
     (effects (font (size 1.27 1.27)) (justify left bottom))
   )
@@
     (effects (font (size 1.27 1.27)) (justify left bottom))
   )
-  (label "DataB2" (at 193.04 99.06 0) (fields_autoplaced)
+  (label "DataB2" (at 193.04 93.98 0) (fields_autoplaced)
     (effects (font (size 1.27 1.27)) (justify left bottom))
   )
@@
     (effects (font (size 1.27 1.27)) (justify right bottom))
   )
-  (label "DataA2" (at 193.04 119.38 0) (fields_autoplaced)
+  (label "DataA2" (at 193.04 114.3 0) (fields_autoplaced)
     (effects (font (size 1.27 1.27)) (justify left bottom))
   )
@@
     (effects (font (size 1.27 1.27)) (justify right bottom))
   )
-  (label "DataA2" (at 193.04 55.88 0) (fields_autoplaced)
+  (label "DataA2" (at 193.04 50.8 0) (fields_autoplaced)
     (effects (font (size 1.27 1.27)) (justify left bottom))
   )
@@
     (effects (font (size 1.27 1.27)) (justify right bottom))
   )
-  (label "DataA0" (at 193.04 114.3 0) (fields_autoplaced)
+  (label "DataA0" (at 193.04 119.38 0) (fields_autoplaced)
     (effects (font (size 1.27 1.27)) (justify left bottom))
   )
@@
     (effects (font (size 1.27 1.27)) (justify left bottom))
   )
-  (label "DataB2" (at 193.04 76.2 0) (fields_autoplaced)
+  (label "DataB2" (at 193.04 71.12 0) (fields_autoplaced)
     (effects (font (size 1.27 1.27)) (justify left bottom))
   )
@@
     (effects (font (size 1.27 1.27)) (justify left bottom))
   )
-  (label "DataIn2" (at 241.3 55.88 180) (fields_autoplaced)
+  (label "DataIn2" (at 241.3 50.8 180) (fields_autoplaced)
     (effects (font (size 1.27 1.27)) (justify right bottom))
   )
@@
     (effects (font (size 1.27 1.27)) (justify right bottom))
   )
-  (label "PixelOut2" (at 241.3 76.2 180) (fields_autoplaced)
+  (label "PixelOut2" (at 241.3 71.12 180) (fields_autoplaced)
     (effects (font (size 1.27 1.27)) (justify right bottom))
   )
@@
     (effects (font (size 1.27 1.27)) (justify right bottom))
   )
-  (label "PixelOut0" (at 241.3 71.12 180) (fields_autoplaced)
+  (label "PixelOut0" (at 241.3 76.2 180) (fields_autoplaced)
     (effects (font (size 1.27 1.27)) (justify right bottom))
   )
@@
     (effects (font (size 1.27 1.27)) (justify left bottom))
   )
-  (label "DataA0" (at 193.04 50.8 0) (fields_autoplaced)
+  (label "DataA0" (at 193.04 55.88 0) (fields_autoplaced)
     (effects (font (size 1.27 1.27)) (justify left bottom))
   )
@@
     (effects (font (size 1.27 1.27)) (justify right bottom))
   )
-  (label "DataB0" (at 193.04 93.98 0) (fields_autoplaced)
+  (label "DataB0" (at 193.04 99.06 0) (fields_autoplaced)
     (effects (font (size 1.27 1.27)) (justify left bottom))
   )
@@
     (effects (font (size 1.27 1.27)) (justify left bottom))
   )
-  (label "DataIn0" (at 241.3 50.8 180) (fields_autoplaced)
-    (effects (font (size 1.27 1.27)) (justify right bottom))
-  )
+  (label "DataIn0" (at 241.3 55.88 180) (fields_autoplaced)
+    (effects (font (size 1.27 1.27)) (justify right bottom))
+  )
