File: memory.kicad_sch (KiCad schematic)
At the start: 11 parts, among them U1 AS7C256A-10, U4 74HC00, U5 74CBT16390, U6 74CBT16390, U9 74CBT16390

Commit message: layout continues...
Parts:
- added D1: LED, symbol Device:LED
- added R12: R, symbol Device:R
Connections:
- net GND: now also R12.2
- net ~{BufSel}: now also D1.2 (A)
- new net: D1.1 (K), R12.1
Changed lines of the file:
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@@
+    (stroke (width 0) (type default))
+  )
+  (wire (pts (xy 205.74 24.13) (xy 205.74 26.67))
     (stroke (width 0) (type default))
   )
@@
   )
   (wire (pts (xy 200.66 50.8) (xy 193.04 50.8))
+    (stroke (width 0) (type default))
+  )
+  (wire (pts (xy 184.15 24.13) (xy 190.5 24.13))
     (stroke (width 0) (type default))
   )
@@
   )
   (label "DataA5" (at 193.04 63.5 0) (fields_autoplaced)
+    (effects (font (size 1.27 1.27)) (justify left bottom))
+  )
+  (label "~{BufSel}" (at 184.15 24.13 0) (fields_autoplaced)
     (effects (font (size 1.27 1.27)) (justify left bottom))
   )
@@
         (path "/b1d8dca2-c863-4452-b293-53802be895cc/197218df-cdff-410d-b6f3-6b97d6088888"
           (reference "#PWR020") (unit 1)
+        )
+      )
+    )
+  )
+  (symbol (lib_id "Device:R") (at 201.93 24.13 90) (unit 1)
+    (in_bom yes) (on_board yes) (dnp no) (fields_autoplaced)
+    (property "Reference" "R12" (at 201.93 17.78 90)
+      (effects (font (size 1.27 1.27)))
+    )
+    (property "Value" "R" (at 201.93 20.32 90)
+      (effects (font (size 1.27 1.27)))
+    )
+    (property "Footprint" "" (at 201.93 25.908 90)
+      (effects (font (size 1.27 1.27)) hide)
+    )
+    (property "Datasheet" "~" (at 201.93 24.13 0)
+      (effects (font (size 1.27 1.27)) hide)
+    )
+    (pin "1")
+    (pin "2")
+    (instances
+      (project "6502gpu"
+        (path "/b1d8dca2-c863-4452-b293-53802be895cc/25d51073-b007-4d3a-a895-244d96d772f9"
+          (reference "R12") (unit 1)
+        )
+        (path "/b1d8dca2-c863-4452-b293-53802be895cc/197218df-cdff-410d-b6f3-6b97d6088888"
+          (reference "R17") (unit 1)
         )
       )
@@
     )
   )
+  (symbol (lib_id "power:GND") (at 205.74 26.67 0) (unit 1)
+    (in_bom yes) (on_board yes) (dnp no) (fields_autoplaced)
+    (property "Reference" "#PWR0106" (at 205.74 33.02 0)
+      (effects (font (size 1.27 1.27)) hide)
+    )
+    (property "Value" "GND" (at 205.74 31.75 0)
+      (effects (font (size 1.27 1.27)))
+    )
+    (property "Footprint" "" (at 205.74 26.67 0)
+      (effects (font (size 1.27 1.27)) hide)
+    )
+    (property "Datasheet" "" (at 205.74 26.67 0)
+      (effects (font (size 1.27 1.27)) hide)
+    )
+    (pin "1")
+    (instances
+      (project "6502gpu"
+        (path "/b1d8dca2-c863-4452-b293-53802be895cc/197218df-cdff-410d-b6f3-6b97d6088888"
+          (reference "#PWR0106") (unit 1)
+        )
+      )
+    )
+  )
   (symbol (lib_id "power:GND") (at 110.49 102.87 0) (unit 1)
     (in_bom yes) (on_board yes) (dnp no) (fields_autoplaced)
@@
         )
       )
+    )
+  )
+  (symbol (lib_id "Device:LED") (at 194.31 24.13 180) (unit 1)
+    (in_bom yes) (on_board yes) (dnp no)
+    (property "Reference" "D1" (at 194.31 17.78 0)
+      (effects (font (size 1.27 1.27)))
+    )
+    (property "Value" "LED" (at 194.31 20.32 0)
+      (effects (font (size 1.27 1.27)))
+    )
+    (property "Footprint" "" (at 194.31 24.13 0)
+      (effects (font (size 1.27 1.27)) hide)
+    )
+    (property "Datasheet" "~" (at 194.31 24.13 0)
+      (effects (font (size 1.27 1.27)) hide)
+    )
+    (pin "1")
+    (pin "2")
+    (instances
+      (project "6502gpu"
+        (path "/b1d8dca2-c863-4452-b293-53802be895cc/25d51073-b007-4d3a-a895-244d96d772f9"
+          (reference "D1") (unit 1)
+        )
+        (path "/b1d8dca2-c863-4452-b293-53802be895cc/197218df-cdff-410d-b6f3-6b97d6088888"
+          (reference "D6") (unit 1)
+        )
+      )
