File: memory.kicad_sch (KiCad schematic)
At the start: 13 parts, among them U1 AS7C256A-10, U4 74HC00, U5 74CBT16390, U6 74CBT16390, U9 74CBT16390

Commit message: Done routing!!
Parts:
- removed D1: LED, symbol Device:LED
- removed R12: R, symbol Device:R
Connections:
- net BufSel: now also U4.12; no longer U4.9
- net GND: now also U4.10, U4.9; no longer U4.12, U4.13
- net WriteMem: now also U4.13; no longer U4.10
- net ~{WeB}: now also U4.11; no longer U4.8
Other:
- moved on the sheet: U4C, U4D
Changed lines of the file:
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@@
   (junction (at 81.28 16.51) (diameter 0) (color 0 0 0 0)
   )
+  (junction (at 81.28 107.95) (diameter 0) (color 0 0 0 0)
+  )
+  (junction (at 91.44 200.66) (diameter 0) (color 0 0 0 0)
+  )
   (junction (at 17.78 110.49) (diameter 0) (color 0 0 0 0)
-  )
-  (junction (at 81.28 107.95) (diameter 0) (color 0 0 0 0)
-  )
-  (junction (at 91.44 200.66) (diameter 0) (color 0 0 0 0)
   )
   (junction (at 31.75 69.85) (diameter 0) (color 0 0 0 0)
@@
     (stroke (width 0) (type default))
   )
-  (wire (pts (xy 205.74 24.13) (xy 205.74 26.67))
-    (stroke (width 0) (type default))
-  )
   (wire (pts (xy 71.12 194.31) (xy 77.47 194.31))
     (stroke (width 0) (type default))
@@
   )
   (wire (pts (xy 200.66 50.8) (xy 193.04 50.8))
-    (stroke (width 0) (type default))
-  )
-  (wire (pts (xy 184.15 24.13) (xy 190.5 24.13))
     (stroke (width 0) (type default))
   )
@@
   )
   (label "DataA5" (at 193.04 63.5 0) (fields_autoplaced)
-    (effects (font (size 1.27 1.27)) (justify left bottom))
-  )
-  (label "~{BufSel}" (at 184.15 24.13 0) (fields_autoplaced)
     (effects (font (size 1.27 1.27)) (justify left bottom))
   )
@@
     )
   )
-  (symbol (lib_id "74xx:74HC00") (at 25.4 107.95 0) (unit 4)
+  (symbol (lib_id "74xx:74HC00") (at 45.72 72.39 0) (unit 4)
     (in_bom yes) (on_board yes) (dnp no)
-    (property "Reference" "U4" (at 25.3917 99.06 0)
-      (effects (font (size 1.27 1.27)))
-    )
-    (property "Value" "74HC00" (at 25.3917 101.6 0)
-      (effects (font (size 1.27 1.27)))
-    )
-    (property "Footprint" "Package_SO:SOIC-14_3.9x8.7mm_P1.27mm" (at 25.4 107.95 0)
-      (effects (font (size 1.27 1.27)) hide)
-    )
-    (property "Datasheet" "http://www.ti.com/lit/gpn/sn74hc00" (at 25.4 107.95 0)
+    (property "Reference" "U4" (at 45.7117 63.5 0)
+      (effects (font (size 1.27 1.27)))
+    )
+    (property "Value" "74HC00" (at 45.7117 66.04 0)
+      (effects (font (size 1.27 1.27)))
+    )
+    (property "Footprint" "Package_SO:SOIC-14_3.9x8.7mm_P1.27mm" (at 45.72 72.39 0)
+      (effects (font (size 1.27 1.27)) hide)
+    )
+    (property "Datasheet" "http://www.ti.com/lit/gpn/sn74hc00" (at 45.72 72.39 0)
       (effects (font (size 1.27 1.27)) hide)
     )
@@
         (path "/b1d8dca2-c863-4452-b293-53802be895cc/197218df-cdff-410d-b6f3-6b97d6088888"
           (reference "#PWR020") (unit 1)
-        )
-      )
-    )
-  )
-  (symbol (lib_id "Device:R") (at 201.93 24.13 90) (unit 1)
-    (in_bom yes) (on_board yes) (dnp no) (fields_autoplaced)
-    (property "Reference" "R12" (at 201.93 17.78 90)
-      (effects (font (size 1.27 1.27)))
-    )
-    (property "Value" "R" (at 201.93 20.32 90)
-      (effects (font (size 1.27 1.27)))
-    )
-    (property "Footprint" "" (at 201.93 25.908 90)
-      (effects (font (size 1.27 1.27)) hide)
-    )
-    (property "Datasheet" "~" (at 201.93 24.13 0)
-      (effects (font (size 1.27 1.27)) hide)
-    )
-    (pin "1")
-    (pin "2")
-    (instances
-      (project "6502gpu"
-        (path "/b1d8dca2-c863-4452-b293-53802be895cc/25d51073-b007-4d3a-a895-244d96d772f9"
-          (reference "R12") (unit 1)
-        )
-        (path "/b1d8dca2-c863-4452-b293-53802be895cc/197218df-cdff-410d-b6f3-6b97d6088888"
-          (reference "R17") (unit 1)
         )
       )
@@
     )
   )
-  (symbol (lib_id "74xx:74HC00") (at 45.72 72.39 0) (unit 3)
+  (symbol (lib_id "74xx:74HC00") (at 25.4 107.95 0) (unit 3)
     (in_bom yes) (on_board yes) (dnp no) (fields_autoplaced)
-    (property "Reference" "U4" (at 45.7117 63.5 0)
-      (effects (font (size 1.27 1.27)))
-    )
-    (property "Value" "74HC00" (at 45.7117 66.04 0)
-      (effects (font (size 1.27 1.27)))
-    )
-    (property "Footprint" "Package_SO:SOIC-14_3.9x8.7mm_P1.27mm" (at 45.72 72.39 0)
-      (effects (font (size 1.27 1.27)) hide)
-    )
-    (property "Datasheet" "http://www.ti.com/lit/gpn/sn74hc00" (at 45.72 72.39 0)
+    (property "Reference" "U4" (at 25.3917 99.06 0)
+      (effects (font (size 1.27 1.27)))
+    )
+    (property "Value" "74HC00" (at 25.3917 101.6 0)
+      (effects (font (size 1.27 1.27)))
+    )
+    (property "Footprint" "Package_SO:SOIC-14_3.9x8.7mm_P1.27mm" (at 25.4 107.95 0)
+      (effects (font (size 1.27 1.27)) hide)
+    )
+    (property "Datasheet" "http://www.ti.com/lit/gpn/sn74hc00" (at 25.4 107.95 0)
       (effects (font (size 1.27 1.27)) hide)
     )
@@
         (path "/b1d8dca2-c863-4452-b293-53802be895cc/197218df-cdff-410d-b6f3-6b97d6088888"
           (reference "#PWR019") (unit 1)
-        )
-      )
-    )
-  )
-  (symbol (lib_id "power:GND") (at 205.74 26.67 0) (unit 1)
-    (in_bom yes) (on_board yes) (dnp no) (fields_autoplaced)
-    (property "Reference" "#PWR0106" (at 205.74 33.02 0)
-      (effects (font (size 1.27 1.27)) hide)
-    )
-    (property "Value" "GND" (at 205.74 31.75 0)
-      (effects (font (size 1.27 1.27)))
-    )
-    (property "Footprint" "" (at 205.74 26.67 0)
-      (effects (font (size 1.27 1.27)) hide)
-    )
-    (property "Datasheet" "" (at 205.74 26.67 0)
-      (effects (font (size 1.27 1.27)) hide)
-    )
-    (pin "1")
-    (instances
-      (project "6502gpu"
-        (path "/b1d8dca2-c863-4452-b293-53802be895cc/197218df-cdff-410d-b6f3-6b97d6088888"
-          (reference "#PWR0106") (unit 1)
         )
       )
@@
         )
       )
-    )
-  )
-  (symbol (lib_id "Device:LED") (at 194.31 24.13 180) (unit 1)
-    (in_bom yes) (on_board yes) (dnp no)
-    (property "Reference" "D1" (at 194.31 17.78 0)
-      (effects (font (size 1.27 1.27)))
-    )
-    (property "Value" "LED" (at 194.31 20.32 0)
-      (effects (font (size 1.27 1.27)))
-    )
-    (property "Footprint" "" (at 194.31 24.13 0)
-      (effects (font (size 1.27 1.27)) hide)
-    )
-    (property "Datasheet" "~" (at 194.31 24.13 0)
-      (effects (font (size 1.27 1.27)) hide)
-    )
-    (pin "1")
-    (pin "2")
-    (instances
-      (project "6502gpu"
-        (path "/b1d8dca2-c863-4452-b293-53802be895cc/25d51073-b007-4d3a-a895-244d96d772f9"
-          (reference "D1") (unit 1)
-        )
-        (path "/b1d8dca2-c863-4452-b293-53802be895cc/197218df-cdff-410d-b6f3-6b97d6088888"
-          (reference "D6") (unit 1)
-        )
-      )

Commit message: begin rev 2... more routing :(
Parts:
- added TP1, TP2, TP3, TP4: TestPoint, TestPoint:TestPoint_Pad_D1.5mm, symbol Connector:TestPoint
- U1: symbol Memory_RAM:KM62256CLP -> custom:AS7C256A-10
Connections:
- net +5V: now also U1.7 (VCC), U1.7 (VCC); no longer U1.28 (VCC), U1.28 (VCC)
- net AddrA0: now also U1.17 (A0); no longer U1.10 (A0)
- net AddrA1: now also U1.16 (A1); no longer U1.9 (A1)
- net AddrA10: now also U1.28 (A10); no longer U1.21 (A10)
- net AddrA11: now also U1.2 (A11); no longer U1.23 (A11)
- net AddrA12: now also U1.9 (A12); no longer U1.2 (A12)
- net AddrA13: now also U1.5 (A13); no longer U1.26 (A13)
- net AddrA14: now also U1.8 (A14); no longer U1.1 (A14)
- net AddrA2: now also U1.15 (A2); no longer U1.8 (A2)
- net AddrA3: now also U1.14 (A3); no longer U1.7 (A3)
- net AddrA4: now also U1.13 (A4); no longer U1.6 (A4)
- net AddrA5: now also U1.12 (A5); no longer U1.5 (A5)
- net AddrA6: now also U1.11 (A6); no longer U1.4 (A6)
- net AddrA7: now also U1.10 (A7); no longer U1.3 (A7)
- net AddrA8: now also U1.4 (A8); no longer U1.25 (A8)
- net AddrA9: now also U1.3 (A9); no longer U1.24 (A9)
- net AddrB0: now also U1.17 (A0); no longer U1.10 (A0)
- net AddrB1: now also U1.16 (A1); no longer U1.9 (A1)
- net AddrB10: now also U1.28 (A10); no longer U1.21 (A10)
- net AddrB11: now also U1.2 (A11); no longer U1.23 (A11)
- net AddrB12: now also U1.9 (A12); no longer U1.2 (A12)
- net AddrB13: now also U1.5 (A13); no longer U1.26 (A13)
- net AddrB14: now also U1.8 (A14); no longer U1.1 (A14)
- net AddrB2: now also U1.15 (A2); no longer U1.8 (A2)
- net AddrB3: now also U1.14 (A3); no longer U1.7 (A3)
- net AddrB4: now also U1.13 (A4); no longer U1.6 (A4)
- net AddrB5: now also U1.12 (A5); no longer U1.5 (A5)
- net AddrB6: now also U1.11 (A6); no longer U1.4 (A6)
- net AddrB7: now also U1.10 (A7); no longer U1.3 (A7)
- net AddrB8: now also U1.4 (A8); no longer U1.25 (A8)
- net AddrB9: now also U1.3 (A9); no longer U1.24 (A9)
- net BufSel: now also U1.1 (~{OE}), TP1.1; no longer U1.22 (~{OE})
- net DataA0: now also U1.18 (I/O0); no longer U1.11 (Q0)
- net DataA1: now also U1.19 (I/O1); no longer U1.12 (Q1)
- net DataA2: now also U1.20 (I/O2); no longer U1.13 (Q2)
- net DataA3: now also U1.22 (I/O3); no longer U1.15 (Q3)
- net DataA4: now also U1.23 (I/O4); no longer U1.16 (Q4)
- net DataA5: now also U1.24 (I/O5); no longer U1.17 (Q5)
- net DataA6: now also U1.25 (I/O6); no longer U1.18 (Q6)
- net DataA7: now also U1.26 (I/O7); no longer U1.19 (Q7)
- net DataB0: now also U1.18 (I/O0); no longer U1.11 (Q0)
- net DataB1: now also U1.19 (I/O1); no longer U1.12 (Q1)
- net DataB2: now also U1.20 (I/O2); no longer U1.13 (Q2)
- net DataB3: now also U1.22 (I/O3); no longer U1.15 (Q3)
- net DataB4: now also U1.23 (I/O4); no longer U1.16 (Q4)
- net DataB5: now also U1.24 (I/O5); no longer U1.17 (Q5)
- net DataB6: now also U1.25 (I/O6); no longer U1.18 (Q6)
- net DataB7: now also U1.26 (I/O7); no longer U1.19 (Q7)
- net GND: now also U1.21 (GND), U1.21 (GND), U1.27 (~{CE}), U1.27 (~{CE}); no longer U1.14 (GND), U1.14 (GND), U1.20 (~{CS}), U1.20 (~{CS})
- net ~{BufSel}: now also U1.1 (~{OE}), TP2.1; no longer U1.22 (~{OE})
- net ~{WeA}: now also U1.6 (~{WE}), TP4.1; no longer U1.27 (~{WE})
- net ~{WeB}: now also U1.6 (~{WE}), TP3.1; no longer U1.27 (~{WE})
Changed lines of the file:
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@@
   (junction (at 17.78 110.49) (diameter 0) (color 0 0 0 0)
   )
+  (junction (at 25.4 69.85) (diameter 0) (color 0 0 0 0)
+  )
   (junction (at 31.75 69.85) (diameter 0) (color 0 0 0 0)
   )
@@
     (stroke (width 0) (type default))
   )
-  (wire (pts (xy 55.88 93.98) (xy 60.96 93.98))
+  (wire (pts (xy 55.88 93.98) (xy 62.23 93.98))
     (stroke (width 0) (type default))
   )
@@
     (stroke (width 0) (type default))
   )
-  (wire (pts (xy 40.64 81.28) (xy 46.99 81.28))
+  (wire (pts (xy 40.64 81.28) (xy 53.34 81.28))
     (stroke (width 0) (type default))
   )
@@
     (stroke (width 0) (type default))
   )
-  (wire (pts (xy 21.59 69.85) (xy 31.75 69.85))
+  (wire (pts (xy 21.59 69.85) (xy 25.4 69.85))
     (stroke (width 0) (type default))
   )
@@
     (stroke (width 0) (type default))
   )
-  (wire (pts (xy 53.34 72.39) (xy 58.42 72.39))
-    (stroke (width 0) (type default))
-  )
   (wire (pts (xy 193.04 76.2) (xy 200.66 76.2))
     (stroke (width 0) (type default))
@@
     (stroke (width 0) (type default))
   )
+  (wire (pts (xy 53.34 72.39) (xy 59.69 72.39))
+    (stroke (width 0) (type default))
+  )
   (wire (pts (xy 106.68 39.37) (xy 97.79 39.37))
     (stroke (width 0) (type default))
@@
     (stroke (width 0) (type default))
   )
+  (wire (pts (xy 25.4 69.85) (xy 31.75 69.85))
+    (stroke (width 0) (type default))
+  )
   (bus (pts (xy 53.34 34.29) (xy 53.34 36.83))
     (stroke (width 0) (type default))
@@
     (effects (font (size 1.27 1.27)) (justify left bottom))
   )
-  (label "~{BufSel}" (at 46.99 81.28 180) (fields_autoplaced)
+  (label "~{BufSel}" (at 52.07 81.28 180) (fields_autoplaced)
     (effects (font (size 1.27 1.27)) (justify right bottom))
   )
@@
     )
   )
-  (symbol (lib_id "Memory_RAM:KM62256CLP") (at 158.75 39.37 0) (unit 1)
+  (symbol (lib_id "custom:AS7C256A-10") (at 158.75 39.37 0) (unit 1)
     (in_bom yes) (on_board yes) (dnp no) (fields_autoplaced)
     (property "Reference" "U1" (at 160.9441 13.97 0)
@@
       (effects (font (size 1.27 1.27)) hide)
     )
-    (pin "14")
-    (pin "28")
+    (pin "21")
+    (pin "7")
     (pin "1")
     (pin "10")
@@
     (pin "12")
     (pin "13")
+    (pin "14")
     (pin "15")
     (pin "16")
@@
     (pin "2")
     (pin "20")
-    (pin "21")
     (pin "22")
     (pin "23")
@@
     (pin "26")
     (pin "27")
+    (pin "28")
     (pin "3")
     (pin "4")
     (pin "5")
     (pin "6")
-    (pin "7")
     (pin "8")
     (pin "9")
@@
     )
   )
-  (symbol (lib_id "Memory_RAM:KM62256CLP") (at 158.75 132.08 0) (unit 1)
+  (symbol (lib_id "custom:AS7C256A-10") (at 158.75 132.08 0) (unit 1)
     (in_bom yes) (on_board yes) (dnp no) (fields_autoplaced)
     (property "Reference" "U1" (at 160.9441 106.68 0)
@@
       (effects (font (size 1.27 1.27)) hide)
     )
-    (pin "14")
-    (pin "28")
+    (pin "21")
+    (pin "7")
     (pin "1")
     (pin "10")
@@
     (pin "12")
     (pin "13")
+    (pin "14")
     (pin "15")
     (pin "16")
@@
     (pin "2")
     (pin "20")
-    (pin "21")
     (pin "22")
     (pin "23")
@@
     (pin "26")
     (pin "27")
+    (pin "28")
     (pin "3")
     (pin "4")
     (pin "5")
     (pin "6")
-    (pin "7")
     (pin "8")
     (pin "9")
@@
     )
   )
+  (symbol (lib_id "Connector:TestPoint") (at 25.4 69.85 0) (unit 1)
+    (in_bom yes) (on_board yes) (dnp no)
+    (property "Reference" "TP1" (at 22.86 64.77 0)
+      (effects (font (size 1.27 1.27)) (justify left))
+    )
+    (property "Value" "TestPoint" (at 27.94 67.818 0)
+      (effects (font (size 1.27 1.27)) (justify left) hide)
+    )
+    (property "Footprint" "TestPoint:TestPoint_Pad_D1.5mm" (at 30.48 69.85 0)
+      (effects (font (size 1.27 1.27)) hide)
+    )
+    (property "Datasheet" "~" (at 30.48 69.85 0)
+      (effects (font (size 1.27 1.27)) hide)
+    )
+    (pin "1")
+    (instances
+      (project "6502fb"
+        (path "/b1d8dca2-c863-4452-b293-53802be895cc/197218df-cdff-410d-b6f3-6b97d6088888"
+          (reference "TP1") (unit 1)
+        )
+      )
+    )
+  )
+  (symbol (lib_id "Connector:TestPoint") (at 59.69 72.39 0) (unit 1)
+    (in_bom yes) (on_board yes) (dnp no)
+    (property "Reference" "TP3" (at 57.15 67.31 0)
+      (effects (font (size 1.27 1.27)) (justify left))
+    )
+    (property "Value" "TestPoint" (at 62.23 70.358 0)
+      (effects (font (size 1.27 1.27)) (justify left) hide)
+    )
+    (property "Footprint" "TestPoint:TestPoint_Pad_D1.5mm" (at 64.77 72.39 0)
+      (effects (font (size 1.27 1.27)) hide)
+    )
+    (property "Datasheet" "~" (at 64.77 72.39 0)
+      (effects (font (size 1.27 1.27)) hide)
+    )
+    (pin "1")
+    (instances
+      (project "6502fb"
+        (path "/b1d8dca2-c863-4452-b293-53802be895cc/197218df-cdff-410d-b6f3-6b97d6088888"
+          (reference "TP3") (unit 1)
+        )
+      )
+    )
+  )
   (symbol (lib_id "power:GND") (at 180.34 62.23 0) (unit 1)
     (in_bom yes) (on_board yes) (dnp no) (fields_autoplaced)
@@
     )
   )
+  (symbol (lib_id "Connector:TestPoint") (at 53.34 81.28 0) (unit 1)
+    (in_bom yes) (on_board yes) (dnp no)
+    (property "Reference" "TP2" (at 50.8 76.2 0)
+      (effects (font (size 1.27 1.27)) (justify left))
+    )
+    (property "Value" "TestPoint" (at 55.88 79.248 0)
+      (effects (font (size 1.27 1.27)) (justify left) hide)
+    )
+    (property "Footprint" "TestPoint:TestPoint_Pad_D1.5mm" (at 58.42 81.28 0)
+      (effects (font (size 1.27 1.27)) hide)
+    )
+    (property "Datasheet" "~" (at 58.42 81.28 0)
+      (effects (font (size 1.27 1.27)) hide)
+    )
+    (pin "1")
+    (instances
+      (project "6502fb"
+        (path "/b1d8dca2-c863-4452-b293-53802be895cc/197218df-cdff-410d-b6f3-6b97d6088888"
+          (reference "TP2") (unit 1)
+        )
+      )
+    )
+  )
   (symbol (lib_id "Device:C") (at 110.49 99.06 0) (unit 1)
     (in_bom yes) (on_board yes) (dnp no) (fields_autoplaced)
@@
         )
       )
+    )
+  )
+  (symbol (lib_id "Connector:TestPoint") (at 62.23 93.98 0) (unit 1)
+    (in_bom yes) (on_board yes) (dnp no)
+    (property "Reference" "TP4" (at 59.69 88.9 0)
+      (effects (font (size 1.27 1.27)) (justify left))
+    )
+    (property "Value" "TestPoint" (at 64.77 91.948 0)
+      (effects (font (size 1.27 1.27)) (justify left) hide)
+    )
+    (property "Footprint" "TestPoint:TestPoint_Pad_D1.5mm" (at 67.31 93.98 0)
+      (effects (font (size 1.27 1.27)) hide)
+    )
+    (property "Datasheet" "~" (at 67.31 93.98 0)
+      (effects (font (size 1.27 1.27)) hide)
+    )
+    (pin "1")
+    (instances
+      (project "6502fb"
+        (path "/b1d8dca2-c863-4452-b293-53802be895cc/197218df-cdff-410d-b6f3-6b97d6088888"
+          (reference "TP4") (unit 1)
+        )
+      )

Commit message: fix HC377 package
Parts:
- TP1, TP2, TP3, TP4: footprint TestPoint:TestPoint_Pad_D1.5mm -> TestPoint:TestPoint_Pad_D1.0mm
Changed lines of the file:
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@@
       (effects (font (size 1.27 1.27)) (justify left) hide)
     )
-    (property "Footprint" "TestPoint:TestPoint_Pad_D1.5mm" (at 30.48 69.85 0)
+    (property "Footprint" "TestPoint:TestPoint_Pad_D1.0mm" (at 30.48 69.85 0)
       (effects (font (size 1.27 1.27)) hide)
     )
@@
       (effects (font (size 1.27 1.27)) (justify left) hide)
     )
-    (property "Footprint" "TestPoint:TestPoint_Pad_D1.5mm" (at 64.77 72.39 0)
+    (property "Footprint" "TestPoint:TestPoint_Pad_D1.0mm" (at 64.77 72.39 0)
       (effects (font (size 1.27 1.27)) hide)
     )
@@
       (effects (font (size 1.27 1.27)) (justify left) hide)
     )
-    (property "Footprint" "TestPoint:TestPoint_Pad_D1.5mm" (at 58.42 81.28 0)
+    (property "Footprint" "TestPoint:TestPoint_Pad_D1.0mm" (at 58.42 81.28 0)
       (effects (font (size 1.27 1.27)) hide)
     )
@@
       (effects (font (size 1.27 1.27)) (justify left) hide)
     )
-    (property "Footprint" "TestPoint:TestPoint_Pad_D1.5mm" (at 67.31 93.98 0)
-      (effects (font (size 1.27 1.27)) hide)
-    )
+    (property "Footprint" "TestPoint:TestPoint_Pad_D1.0mm" (at 67.31 93.98 0)
+      (effects (font (size 1.27 1.27)) hide)
+    )

Commit message: Rev2 work
Connections:
- net AddrA0: now also U5.25 (2B15); no longer U5.33 (1B15)
- net AddrA1: now also U5.23 (2B14); no longer U5.35 (1B14)
- net AddrA10: now also U5.2 (2B1), U6.25 (2B15); no longer U5.50 (1B5), U6.19 (2B11)
- net AddrA11: now also U5.3 (2B2), U6.23 (2B14); no longer U5.52 (1B4), U6.20 (2B12)
- net AddrA12: now also U5.11 (2B7); no longer U5.47 (1B7)
- net AddrA13: now also U5.8 (2B5), U6.19 (2B11); no longer U5.56 (1B1), U6.25 (2B15)
- net AddrA14: now also U5.9 (2B6); no longer U5.49 (1B6)
- net AddrA2: now also U5.22 (2B13); no longer U5.36 (1B13)
- net AddrA3: now also U5.20 (2B12); no longer U5.38 (1B12)
- net AddrA4: now also U5.19 (2B11); no longer U5.39 (1B11)
- net AddrA5: now also U5.17 (2B10); no longer U5.41 (1B10)
- net AddrA6: now also U5.16 (2B9); no longer U5.42 (1B9)
- net AddrA7: now also U5.12 (2B8); no longer U5.46 (1B8)
- net AddrA8: now also U5.6 (2B4), U6.20 (2B12); no longer U5.55 (1B2), U6.23 (2B14)
- net AddrA9: now also U5.5 (2B3); no longer U5.53 (1B3)
- net AddrB0: now also U5.33 (1B15); no longer U5.25 (2B15)
- net AddrB1: now also U5.35 (1B14); no longer U5.23 (2B14)
- net AddrB10: now also U5.56 (1B1), U6.33 (1B15); no longer U5.8 (2B5), U6.39 (1B11)
- net AddrB11: now also U5.55 (1B2), U6.35 (1B14); no longer U5.6 (2B4), U6.38 (1B12)
- net AddrB12: now also U5.47 (1B7); no longer U5.11 (2B7)
- net AddrB13: now also U5.50 (1B5), U6.39 (1B11); no longer U5.2 (2B1), U6.33 (1B15)
- net AddrB14: now also U5.49 (1B6); no longer U5.9 (2B6)
- net AddrB2: now also U5.36 (1B13); no longer U5.22 (2B13)
- net AddrB3: now also U5.38 (1B12); no longer U5.20 (2B12)
- net AddrB4: now also U5.39 (1B11); no longer U5.19 (2B11)
- net AddrB5: now also U5.41 (1B10); no longer U5.17 (2B10)
- net AddrB6: now also U5.42 (1B9); no longer U5.16 (2B9)
- net AddrB7: now also U5.46 (1B8); no longer U5.12 (2B8)
- net AddrB8: now also U5.52 (1B4), U6.38 (1B12); no longer U5.3 (2B2), U6.35 (1B14)
- net AddrB9: now also U5.53 (1B3); no longer U5.5 (2B3)
- net AddrCPU10: now also U5.1 (A1); no longer U5.7 (A5)
- net AddrCPU11: now also U5.54 (A2); no longer U5.51 (A4)
- net AddrCPU13: now also U5.7 (A5); no longer U5.1 (A1)
- net AddrCPU8: now also U5.51 (A4); no longer U5.54 (A2)
- net BufSel: now also U5.29 (~{OE2}); no longer U5.30 (~{OE1})
- net DataA0: now also U9.26 (2B16), U9.46 (1B8); no longer U9.19 (2B11), U9.53 (1B3)
- net DataA1: now also U9.25 (2B15), U9.47 (1B7); no longer U9.17 (2B10), U9.55 (1B2)
- net DataA2: now also U9.23 (2B14), U9.49 (1B6); no longer U9.16 (2B9), U9.56 (1B1)
- net DataA3: now also U9.22 (2B13), U9.50 (1B5); no longer U9.20 (2B12), U9.52 (1B4)
- net DataA4: now also U9.20 (2B12), U9.52 (1B4); no longer U9.22 (2B13), U9.50 (1B5)
- net DataA5: now also U9.19 (2B11), U9.53 (1B3); no longer U9.23 (2B14), U9.49 (1B6)
- net DataA6: now also U9.17 (2B10), U9.55 (1B2); no longer U9.25 (2B15), U9.47 (1B7)
- net DataA7: now also U9.16 (2B9), U9.56 (1B1); no longer U9.26 (2B16), U9.46 (1B8)
- net DataB0: now also U9.12 (2B8), U9.32 (1B16); no longer U9.39 (1B11), U9.5 (2B3)
- net DataB1: now also U9.11 (2B7), U9.33 (1B15); no longer U9.3 (2B2), U9.41 (1B10)
- net DataB2: now also U9.35 (1B14), U9.9 (2B6); no longer U9.2 (2B1), U9.42 (1B9)
- net DataB3: now also U9.36 (1B13), U9.8 (2B5); no longer U9.38 (1B12), U9.6 (2B4)
- net DataB4: now also U9.38 (1B12), U9.6 (2B4); no longer U9.36 (1B13), U9.8 (2B5)
- net DataB5: now also U9.39 (1B11), U9.5 (2B3); no longer U9.35 (1B14), U9.9 (2B6)
- net DataB6: now also U9.3 (2B2), U9.41 (1B10); no longer U9.11 (2B7), U9.33 (1B15)
- net DataB7: now also U9.2 (2B1), U9.42 (1B9); no longer U9.12 (2B8), U9.32 (1B16)
- net DataIn0: now also U9.45 (A8); no longer U9.4 (A3)
- net DataIn1: now also U9.10 (A7); no longer U9.54 (A2)
- net DataIn2: now also U9.48 (A6); no longer U9.1 (A1)
- net DataIn3: now also U9.7 (A5); no longer U9.51 (A4)
- net DataIn4: now also U9.51 (A4); no longer U9.7 (A5)
- net DataIn5: now also U9.4 (A3); no longer U9.48 (A6)
- net DataIn6: now also U9.54 (A2); no longer U9.10 (A7)
- net DataIn7: now also U9.1 (A1); no longer U9.45 (A8)
- net PixelOut0: now also U9.31 (A16); no longer U9.18 (A11)
- net PixelOut1: now also U9.24 (A15); no longer U9.40 (A10)
- net PixelOut2: now also U9.34 (A14); no longer U9.15 (A9)
- net PixelOut3: now also U9.21 (A13); no longer U9.37 (A12)
- net PixelOut4: now also U9.37 (A12); no longer U9.21 (A13)
- net PixelOut5: now also U9.18 (A11); no longer U9.34 (A14)
- net PixelOut6: now also U9.40 (A10); no longer U9.24 (A15)
- net PixelOut7: now also U9.15 (A9); no longer U9.31 (A16)
- net Row2: now also U6.37 (A12); no longer U6.34 (A14)
- net Row4: now also U6.24 (A15); no longer U6.18 (A11)
- net Row5: now also U6.34 (A14); no longer U6.37 (A12)
- net Row7: now also U6.18 (A11); no longer U6.24 (A15)
- net ~{BufSel}: now also U5.30 (~{OE1}); no longer U5.29 (~{OE2})
