File: memory.kicad_sch (KiCad schematic)
At the start: 15 parts, among them U1 AS7C256A-10, U4 74HC00, U5 74CBT16390, U6 74CBT16390, U9 74CBT16390

Commit message: rev2 mostly done now
Parts:
- removed TP1, TP2, TP3, TP4: TestPoint, TestPoint:TestPoint_Pad_D1.0mm, symbol Connector:TestPoint
- added J18: Conn_01x03, Connector_PinHeader_2.54mm:PinHeader_1x03_P2.54mm_Vertical, symbol Connector_Generic:Conn_01x03
Connections:
- net ~{BufSel}: now also J18.1 (Pin_1)
- net ~{WeA}: now also J18.2 (Pin_2)
- net ~{WeB}: now also J18.3 (Pin_3)
Changed lines of the file:
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@@
   (title_block
     (title "6502 Framebuffer: Memory")
+    (rev "2.0")
   )
   (junction (at 91.44 109.22) (diameter 0) (color 0 0 0 0)
@@
   (junction (at 17.78 110.49) (diameter 0) (color 0 0 0 0)
   )
-  (junction (at 25.4 69.85) (diameter 0) (color 0 0 0 0)
-  )
   (junction (at 31.75 69.85) (diameter 0) (color 0 0 0 0)
   )
@@
     (stroke (width 0) (type default))
   )
+  (wire (pts (xy 31.75 125.73) (xy 38.1 125.73))
+    (stroke (width 0) (type default))
+  )
   (wire (pts (xy 106.68 80.01) (xy 97.79 80.01))
     (stroke (width 0) (type default))
@@
     (stroke (width 0) (type default))
   )
-  (wire (pts (xy 55.88 93.98) (xy 62.23 93.98))
+  (wire (pts (xy 55.88 93.98) (xy 59.69 93.98))
     (stroke (width 0) (type default))
   )
@@
     (stroke (width 0) (type default))
   )
-  (wire (pts (xy 40.64 81.28) (xy 53.34 81.28))
+  (wire (pts (xy 40.64 81.28) (xy 48.26 81.28))
     (stroke (width 0) (type default))
   )
@@
     (stroke (width 0) (type default))
   )
-  (wire (pts (xy 21.59 69.85) (xy 25.4 69.85))
+  (wire (pts (xy 21.59 69.85) (xy 31.75 69.85))
     (stroke (width 0) (type default))
   )
@@
     (stroke (width 0) (type default))
   )
+  (wire (pts (xy 31.75 120.65) (xy 38.1 120.65))
+    (stroke (width 0) (type default))
+  )
   (wire (pts (xy 106.68 34.29) (xy 97.79 34.29))
     (stroke (width 0) (type default))
@@
     (stroke (width 0) (type default))
   )
-  (wire (pts (xy 53.34 72.39) (xy 59.69 72.39))
+  (wire (pts (xy 53.34 72.39) (xy 57.15 72.39))
     (stroke (width 0) (type default))
   )
@@
     (stroke (width 0) (type default))
   )
+  (wire (pts (xy 31.75 123.19) (xy 38.1 123.19))
+    (stroke (width 0) (type default))
+  )
   (bus (pts (xy 53.34 24.13) (xy 53.34 26.67))
     (stroke (width 0) (type default))
@@
     (stroke (width 0) (type default))
   )
-  (wire (pts (xy 25.4 69.85) (xy 31.75 69.85))
-    (stroke (width 0) (type default))
-  )
   (bus (pts (xy 53.34 34.29) (xy 53.34 36.83))
     (stroke (width 0) (type default))
@@
     (effects (font (size 1.27 1.27)) (justify right bottom))
   )
+  (label "~{BufSel}" (at 31.75 120.65 0) (fields_autoplaced)
+    (effects (font (size 1.27 1.27)) (justify left bottom))
+  )
   (label "DataA0" (at 179.07 21.59 180) (fields_autoplaced)
     (effects (font (size 1.27 1.27)) (justify right bottom))
@@
     (effects (font (size 1.27 1.27)) (justify left bottom))
   )
-  (label "~{WeA}" (at 60.96 93.98 180) (fields_autoplaced)
+  (label "~{WeA}" (at 59.69 93.98 180) (fields_autoplaced)
     (effects (font (size 1.27 1.27)) (justify right bottom))
   )
@@
     (effects (font (size 1.27 1.27)) (justify left bottom))
   )
-  (label "~{WeB}" (at 58.42 72.39 180) (fields_autoplaced)
+  (label "~{WeB}" (at 57.15 72.39 180) (fields_autoplaced)
     (effects (font (size 1.27 1.27)) (justify right bottom))
   )
@@
     (effects (font (size 1.27 1.27)) (justify right bottom))
   )
+  (label "~{WeA}" (at 31.75 123.19 0) (fields_autoplaced)
+    (effects (font (size 1.27 1.27)) (justify left bottom))
+  )
   (label "AddrB1" (at 137.16 116.84 0) (fields_autoplaced)
     (effects (font (size 1.27 1.27)) (justify left bottom))
@@
     (effects (font (size 1.27 1.27)) (justify left bottom))
   )
-  (label "~{BufSel}" (at 52.07 81.28 180) (fields_autoplaced)
+  (label "~{BufSel}" (at 48.26 81.28 180) (fields_autoplaced)
     (effects (font (size 1.27 1.27)) (justify right bottom))
   )
@@
     (effects (font (size 1.27 1.27)) (justify right bottom))
   )
+  (label "~{WeB}" (at 31.75 125.73 0) (fields_autoplaced)
+    (effects (font (size 1.27 1.27)) (justify left bottom))
+  )
   (label "DataIn4" (at 241.3 58.42 180) (fields_autoplaced)
     (effects (font (size 1.27 1.27)) (justify right bottom))
@@
     )
   )
+  (symbol (lib_id "Connector_Generic:Conn_01x03") (at 43.18 123.19 0) (unit 1)
+    (in_bom yes) (on_board yes) (dnp no) (fields_autoplaced)
+    (property "Reference" "J18" (at 45.72 121.92 0)
+      (effects (font (size 1.27 1.27)) (justify left))
+    )
+    (property "Value" "Conn_01x03" (at 45.72 124.46 0)
+      (effects (font (size 1.27 1.27)) (justify left))
+    )
+    (property "Footprint" "Connector_PinHeader_2.54mm:PinHeader_1x03_P2.54mm_Vertical" (at 43.18 123.19 0)
+      (effects (font (size 1.27 1.27)) hide)
+    )
+    (property "Datasheet" "~" (at 43.18 123.19 0)
+      (effects (font (size 1.27 1.27)) hide)
+    )
+    (pin "1")
+    (pin "2")
+    (pin "3")
+    (instances
+      (project "6502fb"
+        (path "/b1d8dca2-c863-4452-b293-53802be895cc/197218df-cdff-410d-b6f3-6b97d6088888"
+          (reference "J18") (unit 1)
+        )
+      )
+    )
+  )
   (symbol (lib_id "74xx:74HC00") (at 45.72 72.39 0) (unit 4)
     (in_bom yes) (on_board yes) (dnp no)
@@
     )
   )
-  (symbol (lib_id "Connector:TestPoint") (at 25.4 69.85 0) (unit 1)
-    (in_bom yes) (on_board yes) (dnp no)
-    (property "Reference" "TP1" (at 22.86 64.77 0)
-      (effects (font (size 1.27 1.27)) (justify left))
-    )
-    (property "Value" "TestPoint" (at 27.94 67.818 0)
-      (effects (font (size 1.27 1.27)) (justify left) hide)
-    )
-    (property "Footprint" "TestPoint:TestPoint_Pad_D1.0mm" (at 30.48 69.85 0)
-      (effects (font (size 1.27 1.27)) hide)
-    )
-    (property "Datasheet" "~" (at 30.48 69.85 0)
-      (effects (font (size 1.27 1.27)) hide)
-    )
-    (pin "1")
-    (instances
-      (project "6502fb"
-        (path "/b1d8dca2-c863-4452-b293-53802be895cc/197218df-cdff-410d-b6f3-6b97d6088888"
-          (reference "TP1") (unit 1)
-        )
-      )
-    )
-  )
-  (symbol (lib_id "Connector:TestPoint") (at 59.69 72.39 0) (unit 1)
-    (in_bom yes) (on_board yes) (dnp no)
-    (property "Reference" "TP3" (at 57.15 67.31 0)
-      (effects (font (size 1.27 1.27)) (justify left))
-    )
-    (property "Value" "TestPoint" (at 62.23 70.358 0)
-      (effects (font (size 1.27 1.27)) (justify left) hide)
-    )
-    (property "Footprint" "TestPoint:TestPoint_Pad_D1.0mm" (at 64.77 72.39 0)
-      (effects (font (size 1.27 1.27)) hide)
-    )
-    (property "Datasheet" "~" (at 64.77 72.39 0)
-      (effects (font (size 1.27 1.27)) hide)
-    )
-    (pin "1")
-    (instances
-      (project "6502fb"
-        (path "/b1d8dca2-c863-4452-b293-53802be895cc/197218df-cdff-410d-b6f3-6b97d6088888"
-          (reference "TP3") (unit 1)
-        )
-      )
-    )
-  )
   (symbol (lib_id "power:GND") (at 180.34 62.23 0) (unit 1)
     (in_bom yes) (on_board yes) (dnp no) (fields_autoplaced)
@@
     )
   )
-  (symbol (lib_id "Connector:TestPoint") (at 53.34 81.28 0) (unit 1)
-    (in_bom yes) (on_board yes) (dnp no)
-    (property "Reference" "TP2" (at 50.8 76.2 0)
-      (effects (font (size 1.27 1.27)) (justify left))
-    )
-    (property "Value" "TestPoint" (at 55.88 79.248 0)
-      (effects (font (size 1.27 1.27)) (justify left) hide)
-    )
-    (property "Footprint" "TestPoint:TestPoint_Pad_D1.0mm" (at 58.42 81.28 0)
-      (effects (font (size 1.27 1.27)) hide)
-    )
-    (property "Datasheet" "~" (at 58.42 81.28 0)
-      (effects (font (size 1.27 1.27)) hide)
-    )
-    (pin "1")
-    (instances
-      (project "6502fb"
-        (path "/b1d8dca2-c863-4452-b293-53802be895cc/197218df-cdff-410d-b6f3-6b97d6088888"
-          (reference "TP2") (unit 1)
-        )
-      )
-    )
-  )
   (symbol (lib_id "Device:C") (at 110.49 99.06 0) (unit 1)
     (in_bom yes) (on_board yes) (dnp no) (fields_autoplaced)
@@
         )
       )
-    )
-  )
-  (symbol (lib_id "Connector:TestPoint") (at 62.23 93.98 0) (unit 1)
-    (in_bom yes) (on_board yes) (dnp no)
-    (property "Reference" "TP4" (at 59.69 88.9 0)
-      (effects (font (size 1.27 1.27)) (justify left))
-    )
-    (property "Value" "TestPoint" (at 64.77 91.948 0)
-      (effects (font (size 1.27 1.27)) (justify left) hide)
-    )
-    (property "Footprint" "TestPoint:TestPoint_Pad_D1.0mm" (at 67.31 93.98 0)
-      (effects (font (size 1.27 1.27)) hide)
-    )
-    (property "Datasheet" "~" (at 67.31 93.98 0)
-      (effects (font (size 1.27 1.27)) hide)
-    )
-    (pin "1")
-    (instances
-      (project "6502fb"
-        (path "/b1d8dca2-c863-4452-b293-53802be895cc/197218df-cdff-410d-b6f3-6b97d6088888"
-          (reference "TP4") (unit 1)
-        )
-      )
