File: 6502gpu.kicad_sch (KiCad schematic)
At the start: 16 parts, among them J1 Conn_01x02, J15 Conn_01x03, J17 Barrel_Jack, J2 Conn_01x08, J3 Conn_01x02, J4 Conn_01x16, J5 Conn_01x02, J6 Conn_01x03, J7 DE15_Receptacle_HighDensity, J8 Conn_01x08, SW1 SW_SPST, U1 74HC86, U2 74HC00, U3 74LV27, U34 LM7805

Commit message: almost done wiring...
Parts:
- added H1, H2, H3, H4: MountingHole, MountingHole:MountingHole_3.2mm_M3, symbol Mechanical:MountingHole
Connections:
- net AddrCPU5: now also U2.1; no longer U2.12
- net AddrCPU7: now also U2.2; no longer U2.13
- net ConfigReg/NmiEnable: now also U2.13; no longer U2.2
- net VBlank: now also U2.12; no longer U2.1
- net ~{NMI}: now also U2.11; no longer U2.3
- net ~{RegSel}: now also U2.3; no longer U2.11
- net ~{FbSelected} renamed ~{FbSel}
Other:
- moved on the sheet: U2A, U2D
Changed lines of the file:
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@@
     (stroke (width 0) (type default))
   )
-  (wire (pts (xy 191.77 80.01) (xy 201.93 80.01))
+  (wire (pts (xy 194.31 80.01) (xy 201.93 80.01))
     (stroke (width 0) (type default))
   )
@@
     (stroke (width 0) (type default))
   )
-  (wire (pts (xy 201.93 77.47) (xy 191.77 77.47))
+  (wire (pts (xy 201.93 77.47) (xy 194.31 77.47))
     (stroke (width 0) (type default))
   )
@@
     (stroke (width 0) (type default))
   )
-  (wire (pts (xy 201.93 95.25) (xy 191.77 95.25))
+  (wire (pts (xy 201.93 95.25) (xy 194.31 95.25))
     (stroke (width 0) (type default))
   )
@@
     (stroke (width 0) (type default))
   )
-  (wire (pts (xy 191.77 82.55) (xy 201.93 82.55))
+  (wire (pts (xy 194.31 82.55) (xy 201.93 82.55))
     (stroke (width 0) (type default))
   )
@@
     (stroke (width 0) (type default))
   )
-  (wire (pts (xy 191.77 100.33) (xy 201.93 100.33))
+  (wire (pts (xy 194.31 100.33) (xy 201.93 100.33))
     (stroke (width 0) (type default))
   )
@@
     (stroke (width 0) (type default))
   )
-  (wire (pts (xy 201.93 97.79) (xy 191.77 97.79))
+  (wire (pts (xy 201.93 97.79) (xy 194.31 97.79))
     (stroke (width 0) (type default))
   )
@@
     (effects (font (size 1.27 1.27)) (justify right bottom))
   )
-  (label "~{FbSelected}" (at 125.73 148.59 0) (fields_autoplaced)
+  (label "~{FbSel}" (at 125.73 148.59 0) (fields_autoplaced)
     (effects (font (size 1.27 1.27)) (justify left bottom))
   )
@@
     (effects (font (size 1.27 1.27)) (justify right bottom))
   )
-  (label "R~{W}" (at 191.77 80.01 0) (fields_autoplaced)
+  (label "R~{W}" (at 194.31 80.01 0) (fields_autoplaced)
     (effects (font (size 1.27 1.27)) (justify left bottom))
   )
@@
     (effects (font (size 1.27 1.27)) (justify left bottom))
   )
-  (label "R~{W}" (at 191.77 100.33 0) (fields_autoplaced)
+  (label "R~{W}" (at 194.31 100.33 0) (fields_autoplaced)
     (effects (font (size 1.27 1.27)) (justify left bottom))
   )
@@
     (effects (font (size 1.27 1.27)) (justify left bottom))
   )
-  (label "~{FbSelected}" (at 191.77 82.55 0) (fields_autoplaced)
+  (label "~{FbSel}" (at 194.31 82.55 0) (fields_autoplaced)
     (effects (font (size 1.27 1.27)) (justify left bottom))
   )
@@
     (effects (font (size 1.27 1.27)) (justify right bottom))
   )
-  (label "~{FbSelected}" (at 246.38 48.26 180) (fields_autoplaced)
+  (label "~{FbSel}" (at 246.38 48.26 180) (fields_autoplaced)
     (effects (font (size 1.27 1.27)) (justify right bottom))
   )
@@
     (effects (font (size 1.27 1.27)) (justify left bottom))
   )
-  (label "~{Phi2}" (at 191.77 77.47 0) (fields_autoplaced)
+  (label "~{Phi2}" (at 194.31 77.47 0) (fields_autoplaced)
     (effects (font (size 1.27 1.27)) (justify left bottom))
   )
@@
     (effects (font (size 1.27 1.27)) (justify right bottom))
   )
-  (label "~{FbSelected}" (at 191.77 97.79 0) (fields_autoplaced)
+  (label "~{FbSel}" (at 194.31 97.79 0) (fields_autoplaced)
     (effects (font (size 1.27 1.27)) (justify left bottom))
   )
@@
     (effects (font (size 1.27 1.27)) (justify right bottom))
   )
-  (label "~{RegSel}" (at 191.77 95.25 0) (fields_autoplaced)
+  (label "~{RegSel}" (at 194.31 95.25 0) (fields_autoplaced)
     (effects (font (size 1.27 1.27)) (justify left bottom))
   )
@@
         (path "/b1d8dca2-c863-4452-b293-53802be895cc"
           (reference "#PWR05") (unit 1)
+        )
+      )
+    )
+  )
+  (symbol (lib_id "Mechanical:MountingHole") (at 245.11 147.32 0) (unit 1)
+    (in_bom yes) (on_board yes) (dnp no) (fields_autoplaced)
+    (property "Reference" "H3" (at 247.65 146.05 0)
+      (effects (font (size 1.27 1.27)) (justify left))
+    )
+    (property "Value" "MountingHole" (at 247.65 148.59 0)
+      (effects (font (size 1.27 1.27)) (justify left))
+    )
+    (property "Footprint" "MountingHole:MountingHole_3.2mm_M3" (at 245.11 147.32 0)
+      (effects (font (size 1.27 1.27)) hide)
+    )
+    (property "Datasheet" "~" (at 245.11 147.32 0)
+      (effects (font (size 1.27 1.27)) hide)
+    )
+    (instances
+      (project "6502gpu"
+        (path "/b1d8dca2-c863-4452-b293-53802be895cc"
+          (reference "H3") (unit 1)
         )
       )
@@
     )
   )
+  (symbol (lib_id "Mechanical:MountingHole") (at 245.11 140.97 0) (unit 1)
+    (in_bom yes) (on_board yes) (dnp no) (fields_autoplaced)
+    (property "Reference" "H2" (at 247.65 139.7 0)
+      (effects (font (size 1.27 1.27)) (justify left))
+    )
+    (property "Value" "MountingHole" (at 247.65 142.24 0)
+      (effects (font (size 1.27 1.27)) (justify left))
+    )
+    (property "Footprint" "MountingHole:MountingHole_3.2mm_M3" (at 245.11 140.97 0)
+      (effects (font (size 1.27 1.27)) hide)
+    )
+    (property "Datasheet" "~" (at 245.11 140.97 0)
+      (effects (font (size 1.27 1.27)) hide)
+    )
+    (instances
+      (project "6502gpu"
+        (path "/b1d8dca2-c863-4452-b293-53802be895cc"
+          (reference "H2") (unit 1)
+        )
+      )
+    )
+  )
   (symbol (lib_id "Connector_Generic:Conn_01x08") (at 153.67 92.71 0) (unit 1)
     (in_bom yes) (on_board yes) (dnp no) (fields_autoplaced)
@@
     )
   )
+  (symbol (lib_id "Mechanical:MountingHole") (at 245.11 134.62 0) (unit 1)
+    (in_bom yes) (on_board yes) (dnp no) (fields_autoplaced)
+    (property "Reference" "H1" (at 247.65 133.35 0)
+      (effects (font (size 1.27 1.27)) (justify left))
+    )
+    (property "Value" "MountingHole" (at 247.65 135.89 0)
+      (effects (font (size 1.27 1.27)) (justify left))
+    )
+    (property "Footprint" "MountingHole:MountingHole_3.2mm_M3" (at 245.11 134.62 0)
+      (effects (font (size 1.27 1.27)) hide)
+    )
+    (property "Datasheet" "~" (at 245.11 134.62 0)
+      (effects (font (size 1.27 1.27)) hide)
+    )
+    (instances
+      (project "6502gpu"
+        (path "/b1d8dca2-c863-4452-b293-53802be895cc"
+          (reference "H1") (unit 1)
+        )
+      )
+    )
+  )
+  (symbol (lib_id "Mechanical:MountingHole") (at 245.11 153.67 0) (unit 1)
+    (in_bom yes) (on_board yes) (dnp no) (fields_autoplaced)
+    (property "Reference" "H4" (at 247.65 152.4 0)
+      (effects (font (size 1.27 1.27)) (justify left))
+    )
+    (property "Value" "MountingHole" (at 247.65 154.94 0)
+      (effects (font (size 1.27 1.27)) (justify left))
+    )
+    (property "Footprint" "MountingHole:MountingHole_3.2mm_M3" (at 245.11 153.67 0)
+      (effects (font (size 1.27 1.27)) hide)
+    )
+    (property "Datasheet" "~" (at 245.11 153.67 0)
+      (effects (font (size 1.27 1.27)) hide)
+    )
+    (instances
+      (project "6502gpu"
+        (path "/b1d8dca2-c863-4452-b293-53802be895cc"
+          (reference "H4") (unit 1)
+        )
+      )
+    )
+  )
   (symbol (lib_id "Device:C") (at 49.53 44.45 0) (unit 1)
     (in_bom yes) (on_board yes) (dnp no) (fields_autoplaced)
@@
     )
   )
-  (symbol (lib_id "74xx:74HC00") (at 118.11 146.05 0) (unit 1)
+  (symbol (lib_id "74xx:74HC00") (at 111.76 66.04 0) (unit 1)
     (in_bom yes) (on_board yes) (dnp no)
-    (property "Reference" "U2" (at 118.1017 137.16 0)
-      (effects (font (size 1.27 1.27)))
-    )
-    (property "Value" "74HC00" (at 118.1017 139.7 0)
-      (effects (font (size 1.27 1.27)))
-    )
-    (property "Footprint" "Package_SO:SOIC-14_3.9x8.7mm_P1.27mm" (at 118.11 146.05 0)
-      (effects (font (size 1.27 1.27)) hide)
-    )
-    (property "Datasheet" "http://www.ti.com/lit/gpn/sn74hc00" (at 118.11 146.05 0)
+    (property "Reference" "U2" (at 111.7517 57.15 0)
+      (effects (font (size 1.27 1.27)))
+    )
+    (property "Value" "74HC00" (at 111.7517 59.69 0)
+      (effects (font (size 1.27 1.27)))
+    )
+    (property "Footprint" "Package_SO:SOIC-14_3.9x8.7mm_P1.27mm" (at 111.76 66.04 0)
+      (effects (font (size 1.27 1.27)) hide)
+    )
+    (property "Datasheet" "http://www.ti.com/lit/gpn/sn74hc00" (at 111.76 66.04 0)
       (effects (font (size 1.27 1.27)) hide)
     )
@@
     )
   )
-  (symbol (lib_id "74xx:74HC00") (at 111.76 66.04 0) (unit 4)
-    (in_bom yes) (on_board yes) (dnp no) (fields_autoplaced)
-    (property "Reference" "U2" (at 111.7517 57.15 0)
-      (effects (font (size 1.27 1.27)))
-    )
-    (property "Value" "74HC00" (at 111.7517 59.69 0)
-      (effects (font (size 1.27 1.27)))
-    )
-    (property "Footprint" "Package_SO:SOIC-14_3.9x8.7mm_P1.27mm" (at 111.76 66.04 0)
-      (effects (font (size 1.27 1.27)) hide)
-    )
-    (property "Datasheet" "http://www.ti.com/lit/gpn/sn74hc00" (at 111.76 66.04 0)
-      (effects (font (size 1.27 1.27)) hide)
-    )
+  (symbol (lib_id "74xx:74HC00") (at 118.11 146.05 0) (unit 4)
+    (in_bom yes) (on_board yes) (dnp no) (fields_autoplaced)
+    (property "Reference" "U2" (at 118.1017 137.16 0)
+      (effects (font (size 1.27 1.27)))
+    )
+    (property "Value" "74HC00" (at 118.1017 139.7 0)
+      (effects (font (size 1.27 1.27)))
+    )
+    (property "Footprint" "Package_SO:SOIC-14_3.9x8.7mm_P1.27mm" (at 118.11 146.05 0)
+      (effects (font (size 1.27 1.27)) hide)
+    )
+    (property "Datasheet" "http://www.ti.com/lit/gpn/sn74hc00" (at 118.11 146.05 0)
+      (effects (font (size 1.27 1.27)) hide)
+    )

Commit message: Done routing!!
Parts:
- removed J17: Barrel_Jack, Connector_BarrelJack:BarrelJack_CUI_PJ-102AH_Horizontal, symbol Connector:Barrel_Jack_Switch
- removed SW1: SW_SPST, symbol Switch:SW_SPST
- removed U34: LM7805, Package_TO_SOT_THT:TO-220-3_Vertical, symbol Regulator_Linear:LM7805_TO220
Connections:
- net +5V: now also U1.12; no longer U1.9
- net GND: now also U1.10, U1.9; no longer U1.12, U1.13
- net R~{W}: now also U3.10; no longer U3.11
- net WriteMem: now also U3.8; no longer U3.6
- net ~{FbSel}: now also U3.9; no longer U3.10
- net ~{Phi2}: now also U3.11; no longer U3.3
- net ~{RegSel}: now also U3.3; no longer U3.9
- net ~{WriteReg}: now also U1.11; no longer U1.8
- new net: U1.13, U3.6
Other:
- moved on the sheet: U1C, U1D, U3B, U3C
