File: config_reg.kicad_sch (KiCad schematic)
At the start: 2 parts, among them U29 74HC377

Commit message: begin rev 2... more routing :(
Parts:
- added J17: Conn_01x05, Connector_PinHeader_2.54mm:PinHeader_1x05_P2.54mm_Vertical, symbol Connector_Generic:Conn_01x05
Connections:
- net BankSel: now also J17.2 (Pin_2)
- net BlankBlack: now also J17.5 (Pin_5)
- net BlankWhite: now also J17.4 (Pin_4)
- net BufSel: now also J17.1 (Pin_1)
- net NmiEnable: now also J17.3 (Pin_3)
Changed lines of the file:
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@@
+    (stroke (width 0) (type default))
+  )
+  (wire (pts (xy 157.48 90.17) (xy 168.91 90.17))
     (stroke (width 0) (type default))
   )
@@
   )
   (wire (pts (xy 101.6 110.49) (xy 111.76 110.49))
+    (stroke (width 0) (type default))
+  )
+  (wire (pts (xy 157.48 87.63) (xy 168.91 87.63))
     (stroke (width 0) (type default))
   )
@@
     (stroke (width 0) (type default))
   )
+  (wire (pts (xy 157.48 92.71) (xy 168.91 92.71))
+    (stroke (width 0) (type default))
+  )
   (bus (pts (xy 101.6 92.71) (xy 101.6 95.25))
     (stroke (width 0) (type default))
@@
     (stroke (width 0) (type default))
   )
+  (wire (pts (xy 157.48 85.09) (xy 168.91 85.09))
+    (stroke (width 0) (type default))
+  )
   (wire (pts (xy 111.76 95.25) (xy 104.14 95.25))
     (stroke (width 0) (type default))
   )
   (wire (pts (xy 111.76 87.63) (xy 104.14 87.63))
+    (stroke (width 0) (type default))
+  )
+  (wire (pts (xy 157.48 95.25) (xy 168.91 95.25))
     (stroke (width 0) (type default))
   )
@@
     (effects (font (size 1.27 1.27)) (justify left bottom))
   )
+  (label "BankSel" (at 157.48 87.63 0) (fields_autoplaced)
+    (effects (font (size 1.27 1.27)) (justify left bottom))
+  )
   (label "DataIn4" (at 104.14 95.25 0) (fields_autoplaced)
     (effects (font (size 1.27 1.27)) (justify left bottom))
@@
     (effects (font (size 1.27 1.27)) (justify left bottom))
   )
+  (label "BlankWhite" (at 157.48 92.71 0) (fields_autoplaced)
+    (effects (font (size 1.27 1.27)) (justify left bottom))
+  )
+  (label "BufSel" (at 157.48 85.09 0) (fields_autoplaced)
+    (effects (font (size 1.27 1.27)) (justify left bottom))
+  )
+  (label "NmiEnable" (at 157.48 90.17 0) (fields_autoplaced)
+    (effects (font (size 1.27 1.27)) (justify left bottom))
+  )
   (label "DataIn3" (at 104.14 92.71 0) (fields_autoplaced)
+    (effects (font (size 1.27 1.27)) (justify left bottom))
+  )
+  (label "BlankBlack" (at 157.48 95.25 0) (fields_autoplaced)
     (effects (font (size 1.27 1.27)) (justify left bottom))
   )
@@
         )
       )
+    )
+  )
+  (symbol (lib_id "Connector_Generic:Conn_01x05") (at 173.99 90.17 0) (unit 1)
+    (in_bom yes) (on_board yes) (dnp no) (fields_autoplaced)
+    (property "Reference" "J17" (at 176.53 88.9 0)
+      (effects (font (size 1.27 1.27)) (justify left))
+    )
+    (property "Value" "Conn_01x05" (at 176.53 91.44 0)
+      (effects (font (size 1.27 1.27)) (justify left))
+    )
+    (property "Footprint" "Connector_PinHeader_2.54mm:PinHeader_1x05_P2.54mm_Vertical" (at 173.99 90.17 0)
+      (effects (font (size 1.27 1.27)) hide)
+    )
+    (property "Datasheet" "~" (at 173.99 90.17 0)
+      (effects (font (size 1.27 1.27)) hide)
+    )
+    (pin "1")
+    (pin "2")
+    (pin "3")
+    (pin "4")
+    (pin "5")
+    (instances
+      (project "6502fb"
+        (path "/b1d8dca2-c863-4452-b293-53802be895cc/25d51073-b007-4d3a-a895-244d96d772f9"
+          (reference "J17") (unit 1)
+        )
+      )

Commit message: fix HC377 package
Parts:
- U29: footprint Package_SO:SOIC-20W_7.5x12.8mm_P1.27mm -> custom:SOIC-20_5.3x12.6mm_P1.27mm
Changed lines of the file:
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@@
       (effects (font (size 1.27 1.27)) (justify left))
     )
-    (property "Footprint" "Package_SO:SOIC-20W_7.5x12.8mm_P1.27mm" (at 124.46 97.79 0)
+    (property "Footprint" "custom:SOIC-20_5.3x12.6mm_P1.27mm" (at 124.46 97.79 0)
       (effects (font (size 1.27 1.27)) hide)
     )

Commit message: Rev2 work
Connections:
- net BankSel: now also U29.9 (Q3); no longer U29.5 (Q1)
- net BlankBlack: now also U29.2 (Q0); no longer U29.12 (Q4)
- net BlankWhite: now also U29.5 (Q1); no longer U29.9 (Q3)
- net BufSel: now also U29.12 (Q4); no longer U29.2 (Q0)
- net DataIn0: now also U29.13 (D4); no longer U29.3 (D0)
- net DataIn1: now also U29.8 (D3); no longer U29.4 (D1)
- net DataIn3: now also U29.4 (D1); no longer U29.8 (D3)
- net DataIn4: now also U29.3 (D0); no longer U29.13 (D4)
Changed lines of the file:
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@@
     (stroke (width 0) (type default))
   )
-  (wire (pts (xy 111.76 92.71) (xy 104.14 92.71))
+  (wire (pts (xy 111.76 87.63) (xy 104.14 87.63))
     (stroke (width 0) (type default))
   )
@@
     (stroke (width 0) (type default))
   )
-  (wire (pts (xy 111.76 95.25) (xy 104.14 95.25))
+  (wire (pts (xy 111.76 85.09) (xy 104.14 85.09))
     (stroke (width 0) (type default))
   )
-  (wire (pts (xy 111.76 87.63) (xy 104.14 87.63))
+  (wire (pts (xy 111.76 92.71) (xy 104.14 92.71))
     (stroke (width 0) (type default))
   )
@@
     (stroke (width 0) (type default))
   )
-  (wire (pts (xy 111.76 85.09) (xy 104.14 85.09))
+  (wire (pts (xy 111.76 95.25) (xy 104.14 95.25))
     (stroke (width 0) (type default))
   )
@@
     (effects (font (size 1.27 1.27)) (justify left bottom))
   )
-  (label "DataIn1" (at 104.14 87.63 0) (fields_autoplaced)
+  (label "DataIn1" (at 104.14 92.71 0) (fields_autoplaced)
     (effects (font (size 1.27 1.27)) (justify left bottom))
   )
-  (label "DataIn0" (at 104.14 85.09 0) (fields_autoplaced)
+  (label "DataIn0" (at 104.14 95.25 0) (fields_autoplaced)
     (effects (font (size 1.27 1.27)) (justify left bottom))
   )
@@
     (effects (font (size 1.27 1.27)) (justify left bottom))
   )
-  (label "DataIn4" (at 104.14 95.25 0) (fields_autoplaced)
+  (label "DataIn4" (at 104.14 85.09 0) (fields_autoplaced)
     (effects (font (size 1.27 1.27)) (justify left bottom))
   )
@@
     (effects (font (size 1.27 1.27)) (justify left bottom))
   )
-  (label "DataIn3" (at 104.14 92.71 0) (fields_autoplaced)
+  (label "DataIn3" (at 104.14 87.63 0) (fields_autoplaced)
     (effects (font (size 1.27 1.27)) (justify left bottom))
   )
@@
     (effects (font (size 1.27 1.27)) (justify right))
   )
-  (hierarchical_label "BankSel" (shape output) (at 137.16 87.63 0) (fields_autoplaced)
+  (hierarchical_label "BankSel" (shape output) (at 137.16 92.71 0) (fields_autoplaced)
     (effects (font (size 1.27 1.27)) (justify left))
   )
-  (hierarchical_label "BufSel" (shape output) (at 137.16 85.09 0) (fields_autoplaced)
+  (hierarchical_label "BufSel" (shape output) (at 137.16 95.25 0) (fields_autoplaced)
     (effects (font (size 1.27 1.27)) (justify left))
   )
-  (hierarchical_label "BlankBlack" (shape output) (at 137.16 95.25 0) (fields_autoplaced)
+  (hierarchical_label "BlankBlack" (shape output) (at 137.16 85.09 0) (fields_autoplaced)
     (effects (font (size 1.27 1.27)) (justify left))
   )
-  (hierarchical_label "BlankWhite" (shape output) (at 137.16 92.71 0) (fields_autoplaced)
+  (hierarchical_label "BlankWhite" (shape output) (at 137.16 87.63 0) (fields_autoplaced)
     (effects (font (size 1.27 1.27)) (justify left))
   )
