File: 6502fb.kicad_sch (KiCad schematic)
At the start: 17 parts, among them J1 Conn_01x02, J15 Conn_01x03, J2 Conn_01x08, J3 Conn_01x02, J4 Conn_01x16, J5 Conn_01x02, J6 Conn_01x03, J7 DE15_Receptacle_HighDensity, J8 Conn_01x08, U1 74HC86, U2 74HC00, U3 74LV27

Commit message: begin rev 2... more routing :(
Parts:
- J7: footprint Connector_Dsub:DSUB-15-HD_Female_Horizontal_P2.29x1.98mm_EdgePinOffset8.35mm_Housed_MountingHolesOffset10.89mm -> custom:DSUB-15-HD_Female_Horizontal_P2.29x1.98mm_EdgePinOffset8.35mm_Housed_MountingHolesOffset10.89mm
Changed lines of the file:
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@@
       (effects (font (size 1.27 1.27)))
     )
-    (property "Footprint" "Connector_Dsub:DSUB-15-HD_Female_Horizontal_P2.29x1.98mm_EdgePinOffset8.35mm_Housed_MountingHolesOffset10.89mm" (at 168.91 119.38 0)
+    (property "Footprint" "custom:DSUB-15-HD_Female_Horizontal_P2.29x1.98mm_EdgePinOffset8.35mm_Housed_MountingHolesOffset10.89mm" (at 168.91 119.38 0)
       (effects (font (size 1.27 1.27)) hide)
     )

Commit message: Rev2 work
Connections:
- net AddrCPU5: now also U2.2; no longer U2.1
- net AddrCPU7: now also U2.1; no longer U2.2
- net AddrSel: now also U2.13; no longer U2.5
- net ConfigReg/NmiEnable: now also U2.4; no longer U2.13
- net VBlank: now also U2.5; no longer U2.12
- net ~{FbSel}: now also U2.11; no longer U2.6
- net ~{NMI}: now also U2.6; no longer U2.11
- net at U1.3: now also U2.12; no longer U2.4
Other:
- moved on the sheet: U2B, U2D
Changed lines of the file:
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@@
     )
   )
-  (symbol (lib_id "74xx:74HC00") (at 228.6 48.26 0) (unit 2)
-    (in_bom yes) (on_board yes) (dnp no) (fields_autoplaced)
-    (property "Reference" "U2" (at 228.5917 39.37 0)
-      (effects (font (size 1.27 1.27)))
-    )
-    (property "Value" "74HC00" (at 228.5917 41.91 0)
-      (effects (font (size 1.27 1.27)))
-    )
-    (property "Footprint" "Package_SO:SOIC-14_3.9x8.7mm_P1.27mm" (at 228.6 48.26 0)
-      (effects (font (size 1.27 1.27)) hide)
-    )
-    (property "Datasheet" "http://www.ti.com/lit/gpn/sn74hc00" (at 228.6 48.26 0)
+  (symbol (lib_id "74xx:74HC00") (at 118.11 146.05 0) (mirror x) (unit 2)
+    (in_bom yes) (on_board yes) (dnp no)
+    (property "Reference" "U2" (at 118.1017 154.94 0)
+      (effects (font (size 1.27 1.27)))
+    )
+    (property "Value" "74HC00" (at 118.1017 152.4 0)
+      (effects (font (size 1.27 1.27)))
+    )
+    (property "Footprint" "Package_SO:SOIC-14_3.9x8.7mm_P1.27mm" (at 118.11 146.05 0)
+      (effects (font (size 1.27 1.27)) hide)
+    )
+    (property "Datasheet" "http://www.ti.com/lit/gpn/sn74hc00" (at 118.11 146.05 0)
       (effects (font (size 1.27 1.27)) hide)
     )
@@
     )
   )
-  (symbol (lib_id "74xx:74HC00") (at 111.76 66.04 0) (unit 1)
+  (symbol (lib_id "74xx:74HC00") (at 111.76 66.04 0) (mirror x) (unit 1)
     (in_bom yes) (on_board yes) (dnp no)
-    (property "Reference" "U2" (at 111.7517 57.15 0)
-      (effects (font (size 1.27 1.27)))
-    )
-    (property "Value" "74HC00" (at 111.7517 59.69 0)
+    (property "Reference" "U2" (at 111.7517 74.93 0)
+      (effects (font (size 1.27 1.27)))
+    )
+    (property "Value" "74HC00" (at 111.7517 72.39 0)
       (effects (font (size 1.27 1.27)))
     )
@@
     )
   )
-  (symbol (lib_id "74xx:74HC00") (at 118.11 146.05 0) (unit 4)
-    (in_bom yes) (on_board yes) (dnp no) (fields_autoplaced)
-    (property "Reference" "U2" (at 118.1017 137.16 0)
-      (effects (font (size 1.27 1.27)))
-    )
-    (property "Value" "74HC00" (at 118.1017 139.7 0)
-      (effects (font (size 1.27 1.27)))
-    )
-    (property "Footprint" "Package_SO:SOIC-14_3.9x8.7mm_P1.27mm" (at 118.11 146.05 0)
-      (effects (font (size 1.27 1.27)) hide)
-    )
-    (property "Datasheet" "http://www.ti.com/lit/gpn/sn74hc00" (at 118.11 146.05 0)
-      (effects (font (size 1.27 1.27)) hide)
-    )
+  (symbol (lib_id "74xx:74HC00") (at 228.6 48.26 0) (unit 4)
+    (in_bom yes) (on_board yes) (dnp no) (fields_autoplaced)
+    (property "Reference" "U2" (at 228.5917 39.37 0)
+      (effects (font (size 1.27 1.27)))
+    )
+    (property "Value" "74HC00" (at 228.5917 41.91 0)
+      (effects (font (size 1.27 1.27)))
+    )
+    (property "Footprint" "Package_SO:SOIC-14_3.9x8.7mm_P1.27mm" (at 228.6 48.26 0)
+      (effects (font (size 1.27 1.27)) hide)
+    )
+    (property "Datasheet" "http://www.ti.com/lit/gpn/sn74hc00" (at 228.6 48.26 0)
+      (effects (font (size 1.27 1.27)) hide)
+    )

Commit message: rev2 mostly done now
Parts:
- removed C35: 10u, Capacitor_SMD:C_1206_3216Metric_Pad1.33x1.80mm_HandSolder, symbol Device:C
- removed J3: Conn_01x02, Connector_PinHeader_2.54mm:PinHeader_1x02_P2.54mm_Vertical, symbol Connector_Generic:Conn_01x02
Connections:
- net +5V: now also U1.1; no longer U1.12
- net AddrPhys14: now also U1.13; no longer U1.1
- net AddrPhys15: now also U1.12; no longer U1.2
- net ~{WriteReg}: now also U1.3; no longer U1.11
- net at U3.6: now also U1.2; no longer U1.13
- net at U2.12: now also U1.11; no longer U1.3
Other:
- moved on the sheet: U1A, U1D
Changed lines of the file:
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@@
   (title_block
     (title "6502 Framebuffer")
+    (rev "2.0")
   )
   (junction (at 177.8 137.16) (diameter 0) (color 0 0 0 0)
@@
   (junction (at 110.49 127) (diameter 0) (color 0 0 0 0)
   )
-  (junction (at 41.91 43.18) (diameter 0) (color 0 0 0 0)
-  )
   (junction (at 90.17 93.98) (diameter 0) (color 0 0 0 0)
   )
-  (junction (at 34.29 45.72) (diameter 0) (color 0 0 0 0)
-  )
   (junction (at 177.8 139.7) (diameter 0) (color 0 0 0 0)
   )
-  (junction (at 34.29 43.18) (diameter 0) (color 0 0 0 0)
+  (junction (at 205.74 48.26) (diameter 0) (color 0 0 0 0)
   )
   (junction (at 177.8 121.92) (diameter 0) (color 0 0 0 0)
@@
   (junction (at 170.18 129.54) (diameter 0) (color 0 0 0 0)
   )
-  (junction (at 205.74 48.26) (diameter 0) (color 0 0 0 0)
-  )
   (junction (at 43.18 96.52) (diameter 0) (color 0 0 0 0)
   )
@@
   )
   (junction (at 177.8 127) (diameter 0) (color 0 0 0 0)
-  )
-  (junction (at 41.91 45.72) (diameter 0) (color 0 0 0 0)
   )
   (no_connect (at 200.66 124.46))
@@
     (stroke (width 0) (type default))
   )
-  (wire (pts (xy 44.45 48.26) (xy 49.53 48.26))
-    (stroke (width 0) (type default))
-  )
   (wire (pts (xy 194.31 80.01) (xy 201.93 80.01))
     (stroke (width 0) (type default))
@@
     (stroke (width 0) (type default))
   )
-  (wire (pts (xy 44.45 45.72) (xy 44.45 48.26))
-    (stroke (width 0) (type default))
-  )
   (wire (pts (xy 55.88 29.21) (xy 60.96 29.21))
     (stroke (width 0) (type default))
@@
     (stroke (width 0) (type default))
   )
-  (wire (pts (xy 41.91 45.72) (xy 44.45 45.72))
-    (stroke (width 0) (type default))
-  )
   (wire (pts (xy 148.59 85.09) (xy 138.43 85.09))
     (stroke (width 0) (type default))
   )
-  (wire (pts (xy 34.29 43.18) (xy 41.91 43.18))
-    (stroke (width 0) (type default))
-  )
   (wire (pts (xy 76.2 73.66) (xy 87.63 73.66))
     (stroke (width 0) (type default))
@@
     (stroke (width 0) (type default))
   )
-  (wire (pts (xy 44.45 40.64) (xy 44.45 43.18))
-    (stroke (width 0) (type default))
-  )
   (bus (pts (xy 90.17 73.66) (xy 90.17 76.2))
     (stroke (width 0) (type default))
@@
     (stroke (width 0) (type default))
   )
-  (wire (pts (xy 34.29 45.72) (xy 41.91 45.72))
-    (stroke (width 0) (type default))
-  )
   (wire (pts (xy 115.57 101.6) (xy 106.68 101.6))
     (stroke (width 0) (type default))
@@
     (stroke (width 0) (type default))
   )
-  (wire (pts (xy 44.45 43.18) (xy 41.91 43.18))
-    (stroke (width 0) (type default))
-  )
   (wire (pts (xy 33.02 83.82) (xy 40.64 83.82))
     (stroke (width 0) (type default))
@@
   )
   (wire (pts (xy 220.98 59.69) (xy 200.66 59.69))
-    (stroke (width 0) (type default))
-  )
-  (wire (pts (xy 49.53 40.64) (xy 44.45 40.64))
     (stroke (width 0) (type default))
   )
@@
     )
   )
-  (symbol (lib_id "power:PWR_FLAG") (at 41.91 43.18 0) (unit 1)
-    (in_bom yes) (on_board yes) (dnp no) (fields_autoplaced)
-    (property "Reference" "#FLG01" (at 41.91 41.275 0)
-      (effects (font (size 1.27 1.27)) hide)
-    )
-    (property "Value" "PWR_FLAG" (at 41.91 38.1 0)
-      (effects (font (size 1.27 1.27)))
-    )
-    (property "Footprint" "" (at 41.91 43.18 0)
-      (effects (font (size 1.27 1.27)) hide)
-    )
-    (property "Datasheet" "~" (at 41.91 43.18 0)
-      (effects (font (size 1.27 1.27)) hide)
-    )
-    (pin "1")
-    (instances
-      (project "6502fb"
-        (path "/b1d8dca2-c863-4452-b293-53802be895cc"
-          (reference "#FLG01") (unit 1)
-        )
-      )
-    )
-  )
-  (symbol (lib_id "74xx:74HC86") (at 224.79 95.25 0) (unit 4)
-    (in_bom yes) (on_board yes) (dnp no) (fields_autoplaced)
-    (property "Reference" "U1" (at 224.4852 86.36 0)
-      (effects (font (size 1.27 1.27)))
-    )
-    (property "Value" "74HC86" (at 224.4852 88.9 0)
-      (effects (font (size 1.27 1.27)))
-    )
-    (property "Footprint" "Package_SO:SOIC-14_3.9x8.7mm_P1.27mm" (at 224.79 95.25 0)
-      (effects (font (size 1.27 1.27)) hide)
-    )
-    (property "Datasheet" "http://www.ti.com/lit/gpn/sn74HC86" (at 224.79 95.25 0)
+  (symbol (lib_id "74xx:74HC86") (at 213.36 45.72 0) (mirror x) (unit 4)
+    (in_bom yes) (on_board yes) (dnp no)
+    (property "Reference" "U1" (at 213.0552 54.61 0)
+      (effects (font (size 1.27 1.27)))
+    )
+    (property "Value" "74HC86" (at 213.0552 52.07 0)
+      (effects (font (size 1.27 1.27)))
+    )
+    (property "Footprint" "Package_SO:SOIC-14_3.9x8.7mm_P1.27mm" (at 213.36 45.72 0)
+      (effects (font (size 1.27 1.27)) hide)
+    )
+    (property "Datasheet" "http://www.ti.com/lit/gpn/sn74HC86" (at 213.36 45.72 0)
       (effects (font (size 1.27 1.27)) hide)
     )
@@
     )
   )
-  (symbol (lib_id "Connector_Generic:Conn_01x02") (at 29.21 43.18 0) (mirror y) (unit 1)
-    (in_bom yes) (on_board yes) (dnp no)
-    (property "Reference" "J3" (at 21.59 43.18 0)
-      (effects (font (size 1.27 1.27)))
-    )
-    (property "Value" "Conn_01x02" (at 21.59 45.72 0)
-      (effects (font (size 1.27 1.27)))
-    )
-    (property "Footprint" "Connector_PinHeader_2.54mm:PinHeader_1x02_P2.54mm_Vertical" (at 29.21 43.18 0)
-      (effects (font (size 1.27 1.27)) hide)
-    )
-    (property "Datasheet" "~" (at 29.21 43.18 0)
-      (effects (font (size 1.27 1.27)) hide)
-    )
-    (pin "1")
-    (pin "2")
-    (instances
-      (project "6502fb"
-        (path "/b1d8dca2-c863-4452-b293-53802be895cc"
-          (reference "J3") (unit 1)
-        )
-      )
-    )
-  )
-  (symbol (lib_id "power:+5V") (at 34.29 43.18 0) (unit 1)
-    (in_bom yes) (on_board yes) (dnp no) (fields_autoplaced)
-    (property "Reference" "#PWR02" (at 34.29 46.99 0)
-      (effects (font (size 1.27 1.27)) hide)
-    )
-    (property "Value" "+5V" (at 34.29 38.1 0)
-      (effects (font (size 1.27 1.27)))
-    )
-    (property "Footprint" "" (at 34.29 43.18 0)
-      (effects (font (size 1.27 1.27)) hide)
-    )
-    (property "Datasheet" "" (at 34.29 43.18 0)
-      (effects (font (size 1.27 1.27)) hide)
-    )
-    (pin "1")
-    (instances
-      (project "6502fb"
-        (path "/b1d8dca2-c863-4452-b293-53802be895cc"
-          (reference "#PWR02") (unit 1)
-        )
-      )
-    )
-  )
-  (symbol (lib_id "power:GND") (at 34.29 45.72 0) (unit 1)
-    (in_bom yes) (on_board yes) (dnp no) (fields_autoplaced)
-    (property "Reference" "#PWR03" (at 34.29 52.07 0)
-      (effects (font (size 1.27 1.27)) hide)
-    )
-    (property "Value" "GND" (at 34.29 50.8 0)
-      (effects (font (size 1.27 1.27)))
-    )
-    (property "Footprint" "" (at 34.29 45.72 0)
-      (effects (font (size 1.27 1.27)) hide)
-    )
-    (property "Datasheet" "" (at 34.29 45.72 0)
-      (effects (font (size 1.27 1.27)) hide)
-    )
-    (pin "1")
-    (instances
-      (project "6502fb"
-        (path "/b1d8dca2-c863-4452-b293-53802be895cc"
-          (reference "#PWR03") (unit 1)
-        )
-      )
-    )
-  )
   (symbol (lib_id "Mechanical:MountingHole") (at 245.11 134.62 0) (unit 1)
     (in_bom yes) (on_board yes) (dnp no) (fields_autoplaced)
@@
     )
   )
-  (symbol (lib_id "Device:C") (at 49.53 44.45 0) (unit 1)
+  (symbol (lib_id "74xx:74HC86") (at 224.79 95.25 0) (unit 1)
     (in_bom yes) (on_board yes) (dnp no) (fields_autoplaced)
-    (property "Reference" "C35" (at 53.34 43.18 0)
-      (effects (font (size 1.27 1.27)) (justify left))
-    )
-    (property "Value" "10u" (at 53.34 45.72 0)
-      (effects (font (size 1.27 1.27)) (justify left))
-    )
-    (property "Footprint" "Capacitor_SMD:C_1206_3216Metric_Pad1.33x1.80mm_HandSolder" (at 50.4952 48.26 0)
-      (effects (font (size 1.27 1.27)) hide)
-    )
-    (property "Datasheet" "~" (at 49.53 44.45 0)
-      (effects (font (size 1.27 1.27)) hide)
-    )
-    (pin "1")
-    (pin "2")
-    (instances
-      (project "6502fb"
-        (path "/b1d8dca2-c863-4452-b293-53802be895cc"
-          (reference "C35") (unit 1)
-        )
-      )
-    )
-  )
-  (symbol (lib_id "74xx:74HC86") (at 213.36 45.72 0) (unit 1)
-    (in_bom yes) (on_board yes) (dnp no) (fields_autoplaced)
-    (property "Reference" "U1" (at 213.0552 36.83 0)
-      (effects (font (size 1.27 1.27)))
-    )
-    (property "Value" "74HC86" (at 213.0552 39.37 0)
-      (effects (font (size 1.27 1.27)))
-    )
-    (property "Footprint" "Package_SO:SOIC-14_3.9x8.7mm_P1.27mm" (at 213.36 45.72 0)
-      (effects (font (size 1.27 1.27)) hide)
-    )
-    (property "Datasheet" "http://www.ti.com/lit/gpn/sn74HC86" (at 213.36 45.72 0)
+    (property "Reference" "U1" (at 224.4852 86.36 0)
+      (effects (font (size 1.27 1.27)))
+    )
+    (property "Value" "74HC86" (at 224.4852 88.9 0)
+      (effects (font (size 1.27 1.27)))
+    )
+    (property "Footprint" "Package_SO:SOIC-14_3.9x8.7mm_P1.27mm" (at 224.79 95.25 0)
+      (effects (font (size 1.27 1.27)) hide)
+    )
+    (property "Datasheet" "http://www.ti.com/lit/gpn/sn74HC86" (at 224.79 95.25 0)
       (effects (font (size 1.27 1.27)) hide)
     )
@@
         )
       )
-    )
-  )
-  (symbol (lib_id "power:PWR_FLAG") (at 41.91 45.72 0) (mirror x) (unit 1)
-    (in_bom yes) (on_board yes) (dnp no) (fields_autoplaced)
-    (property "Reference" "#FLG02" (at 41.91 47.625 0)
-      (effects (font (size 1.27 1.27)) hide)
-    )
-    (property "Value" "PWR_FLAG" (at 41.91 50.8 0)
-      (effects (font (size 1.27 1.27)))
-    )
-    (property "Footprint" "" (at 41.91 45.72 0)
-      (effects (font (size 1.27 1.27)) hide)
-    )
-    (property "Datasheet" "~" (at 41.91 45.72 0)
-      (effects (font (size 1.27 1.27)) hide)
-    )
-    (pin "1")
-    (instances
-      (project "6502fb"
-        (path "/b1d8dca2-c863-4452-b293-53802be895cc"
-          (reference "#FLG02") (unit 1)
-        )
-      )
