File: counters.kicad_sch (KiCad schematic)
At the start: 34 parts, among them J10 Conn_01x10, J11 Conn_01x03, J12 Conn_01x03, J13 Conn_01x03, J14 Conn_01x03, J16 Conn_01x01, J9 Conn_01x10, U10 74AHC30, U11 74AHC30, U12 74AHC30, U13 74AHC30, U14 74LV163, U15 74LV04, U16 74AC109, U17 74LV163, U18 74LV04, U19 74LV08, U20 74LV163, U21 74AHC30, U22 74AHC30, U23 74AHC30, U24 74AHC30, U25 74AC109, U26 74LV163, U27 74LV163, U28 74LV163, X1 25.175MHz

Commit message: Make DRC quiet, add loooots of vias
Parts:
- U10, U11, U12, U13, U21, U22, U23, U24: symbol 74xx:74LS30 -> custom:74AHC30
Changed lines of the file:
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@@
     )
   )
-  (symbol (lib_id "74xx:74LS30") (at 30.48 88.9 0) (unit 1)
+  (symbol (lib_id "custom:74AHC30") (at 30.48 88.9 0) (unit 1)
     (in_bom yes) (on_board yes) (dnp no) (fields_autoplaced)
     (property "Reference" "U10" (at 30.4717 76.2 0)
@@
     (pin "14")
     (pin "7")
+    (pin "10")
+    (pin "13")
+    (pin "9")
     (instances
       (project "6502gpu"
@@
     )
   )
-  (symbol (lib_id "74xx:74LS30") (at 30.48 138.43 0) (unit 1)
+  (symbol (lib_id "custom:74AHC30") (at 30.48 138.43 0) (unit 1)
     (in_bom yes) (on_board yes) (dnp no) (fields_autoplaced)
     (property "Reference" "U12" (at 30.4717 125.73 0)
@@
     (pin "14")
     (pin "7")
+    (pin "10")
+    (pin "13")
+    (pin "9")
     (instances
       (project "6502gpu"
@@
     )
   )
-  (symbol (lib_id "74xx:74LS30") (at 30.48 162.56 0) (unit 1)
+  (symbol (lib_id "custom:74AHC30") (at 30.48 162.56 0) (unit 1)
     (in_bom yes) (on_board yes) (dnp no) (fields_autoplaced)
     (property "Reference" "U13" (at 30.4717 149.86 0)
@@
     (pin "14")
     (pin "7")
+    (pin "10")
+    (pin "13")
+    (pin "9")
     (instances
       (project "6502gpu"
@@
     )
   )
-  (symbol (lib_id "74xx:74LS30") (at 124.46 143.51 0) (unit 1)
+  (symbol (lib_id "custom:74AHC30") (at 124.46 143.51 0) (unit 1)
     (in_bom yes) (on_board yes) (dnp no)
     (property "Reference" "U23" (at 124.4517 130.81 0)
@@
     (pin "14")
     (pin "7")
+    (pin "10")
+    (pin "13")
+    (pin "9")
     (instances
       (project "6502gpu"
@@
     )
   )
-  (symbol (lib_id "74xx:74LS30") (at 30.48 113.03 0) (unit 1)
+  (symbol (lib_id "custom:74AHC30") (at 30.48 113.03 0) (unit 1)
     (in_bom yes) (on_board yes) (dnp no) (fields_autoplaced)
     (property "Reference" "U11" (at 30.4717 100.33 0)
@@
     (pin "14")
     (pin "7")
+    (pin "10")
+    (pin "13")
+    (pin "9")
     (instances
       (project "6502gpu"
@@
     )
   )
-  (symbol (lib_id "74xx:74LS30") (at 124.46 92.71 0) (unit 1)
+  (symbol (lib_id "custom:74AHC30") (at 124.46 92.71 0) (unit 1)
     (in_bom yes) (on_board yes) (dnp no) (fields_autoplaced)
     (property "Reference" "U21" (at 124.4517 80.01 0)
@@
     (pin "14")
     (pin "7")
+    (pin "10")
+    (pin "13")
+    (pin "9")
     (instances
       (project "6502gpu"
@@
     )
   )
-  (symbol (lib_id "74xx:74LS30") (at 124.46 116.84 0) (unit 1)
+  (symbol (lib_id "custom:74AHC30") (at 124.46 116.84 0) (unit 1)
     (in_bom yes) (on_board yes) (dnp no) (fields_autoplaced)
     (property "Reference" "U22" (at 124.4517 104.14 0)
@@
     (pin "14")
     (pin "7")
+    (pin "10")
+    (pin "13")
+    (pin "9")
     (instances
       (project "6502gpu"
@@
     )
   )
-  (symbol (lib_id "74xx:74LS30") (at 124.46 168.91 0) (unit 1)
+  (symbol (lib_id "custom:74AHC30") (at 124.46 168.91 0) (unit 1)
     (in_bom yes) (on_board yes) (dnp no) (fields_autoplaced)
     (property "Reference" "U24" (at 124.4517 156.21 0)
@@
     (pin "14")
     (pin "7")
-    (instances
-      (project "6502gpu"
+    (pin "10")
+    (pin "13")
+    (pin "9")
+    (instances
+      (project "6502gpu"
