File: dac.kicad_sch (KiCad schematic)
At the start: 4 parts, among them U15 74LV32, U17 74LV32, U30 74LV08, U31 74LS08

Commit message: cleanup
Changed lines of the file:
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@@
     (stroke (width 0) (type default))
   )
-  (wire (pts (xy 62.23 123.19) (xy 73.66 123.19))
+  (wire (pts (xy 60.96 125.73) (xy 73.66 125.73))
     (stroke (width 0) (type default))
   )
   (wire (pts (xy 96.52 125.73) (xy 93.98 125.73))
+    (stroke (width 0) (type default))
+  )
+  (wire (pts (xy 73.66 125.73) (xy 73.66 123.19))
     (stroke (width 0) (type default))
   )
@@
   )
   (wire (pts (xy 91.44 78.74) (xy 96.52 78.74))
+    (stroke (width 0) (type default))
+  )
+  (wire (pts (xy 93.98 128.27) (xy 93.98 125.73))
     (stroke (width 0) (type default))
   )
@@
     (stroke (width 0) (type default))
   )
-  (wire (pts (xy 62.23 125.73) (xy 93.98 125.73))
+  (wire (pts (xy 60.96 128.27) (xy 93.98 128.27))
     (stroke (width 0) (type default))
   )
@@
     (effects (font (size 1.27 1.27)) (justify left bottom))
   )
-  (label "~{ShowBlack}" (at 62.23 125.73 0) (fields_autoplaced)
+  (label "~{ShowBlack}" (at 60.96 128.27 0) (fields_autoplaced)
     (effects (font (size 1.27 1.27)) (justify left bottom))
   )
@@
     (effects (font (size 1.27 1.27)) (justify left bottom))
   )
-  (label "ShowWhite" (at 62.23 123.19 0) (fields_autoplaced)
+  (label "ShowWhite" (at 60.96 125.73 0) (fields_autoplaced)
     (effects (font (size 1.27 1.27)) (justify left bottom))
   )
@@
     (effects (font (size 1.27 1.27)) (justify left bottom))
   )
+  (hierarchical_label "Blue" (shape output) (at 227.33 96.52 0) (fields_autoplaced)
+    (effects (font (size 1.27 1.27)) (justify left))
+  )
   (hierarchical_label "Pixel" (shape input) (at 67.31 120.65 180) (fields_autoplaced)
     (effects (font (size 1.27 1.27)) (justify right))
+  )
+  (hierarchical_label "Red" (shape output) (at 227.33 91.44 0) (fields_autoplaced)
+    (effects (font (size 1.27 1.27)) (justify left))
   )
   (hierarchical_label "HBlank" (shape input) (at 40.64 138.43 180) (fields_autoplaced)
@@
     (effects (font (size 1.27 1.27)) (justify right))
   )
+  (hierarchical_label "Green" (shape output) (at 227.33 93.98 0) (fields_autoplaced)
+    (effects (font (size 1.27 1.27)) (justify left))
+  )
   (symbol (lib_id "74xx:74LS32") (at 83.82 92.71 0) (unit 2)

Commit message: remove 3390, cleanup
Connections:
- net D0 renamed PixelOut0
- net D1 renamed PixelOut1
- net D2 renamed PixelOut2
- net D3 renamed PixelOut3
- net D4 renamed PixelOut4
- net D5 renamed PixelOut5
- net D6 renamed PixelOut6
- net D7 renamed PixelOut7
Changed lines of the file:
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@@
   (junction (at 93.98 55.88) (diameter 0) (color 0 0 0 0)
   )
-  (bus_entry (at 69.85 62.23) (size -2.54 2.54)
-    (stroke (width 0) (type default))
-  )
-  (bus_entry (at 69.85 34.29) (size -2.54 2.54)
-    (stroke (width 0) (type default))
-  )
-  (bus_entry (at 69.85 118.11) (size -2.54 2.54)
-    (stroke (width 0) (type default))
-  )
-  (bus_entry (at 69.85 48.26) (size -2.54 2.54)
-    (stroke (width 0) (type default))
-  )
-  (bus_entry (at 69.85 20.32) (size -2.54 2.54)
-    (stroke (width 0) (type default))
-  )
-  (bus_entry (at 69.85 104.14) (size -2.54 2.54)
-    (stroke (width 0) (type default))
-  )
-  (bus_entry (at 69.85 76.2) (size -2.54 2.54)
-    (stroke (width 0) (type default))
-  )
-  (bus_entry (at 69.85 90.17) (size -2.54 2.54)
-    (stroke (width 0) (type default))
-  )
-  (wire (pts (xy 69.85 62.23) (xy 76.2 62.23))
-    (stroke (width 0) (type default))
-  )
-  (wire (pts (xy 69.85 90.17) (xy 76.2 90.17))
+  (bus_entry (at 62.23 62.23) (size -2.54 2.54)
+    (stroke (width 0) (type default))
+  )
+  (bus_entry (at 62.23 34.29) (size -2.54 2.54)
+    (stroke (width 0) (type default))
+  )
+  (bus_entry (at 62.23 118.11) (size -2.54 2.54)
+    (stroke (width 0) (type default))
+  )
+  (bus_entry (at 62.23 48.26) (size -2.54 2.54)
+    (stroke (width 0) (type default))
+  )
+  (bus_entry (at 62.23 20.32) (size -2.54 2.54)
+    (stroke (width 0) (type default))
+  )
+  (bus_entry (at 62.23 104.14) (size -2.54 2.54)
+    (stroke (width 0) (type default))
+  )
+  (bus_entry (at 62.23 76.2) (size -2.54 2.54)
+    (stroke (width 0) (type default))
+  )
+  (bus_entry (at 62.23 90.17) (size -2.54 2.54)
+    (stroke (width 0) (type default))
+  )
+  (wire (pts (xy 62.23 62.23) (xy 76.2 62.23))
     (stroke (width 0) (type default))
   )
@@
     (stroke (width 0) (type default))
   )
-  (bus (pts (xy 67.31 106.68) (xy 67.31 120.65))
+  (wire (pts (xy 62.23 118.11) (xy 76.2 118.11))
+    (stroke (width 0) (type default))
+  )
+  (bus (pts (xy 59.69 106.68) (xy 59.69 120.65))
+    (stroke (width 0) (type default))
+  )
+  (wire (pts (xy 62.23 90.17) (xy 76.2 90.17))
     (stroke (width 0) (type default))
   )
@@
     (stroke (width 0) (type default))
   )
-  (bus (pts (xy 67.31 92.71) (xy 67.31 106.68))
+  (bus (pts (xy 59.69 92.71) (xy 59.69 106.68))
     (stroke (width 0) (type default))
   )
@@
     (stroke (width 0) (type default))
   )
-  (bus (pts (xy 67.31 64.77) (xy 67.31 78.74))
+  (bus (pts (xy 59.69 64.77) (xy 59.69 78.74))
     (stroke (width 0) (type default))
   )
@@
     (stroke (width 0) (type default))
   )
-  (bus (pts (xy 67.31 36.83) (xy 67.31 50.8))
+  (bus (pts (xy 59.69 36.83) (xy 59.69 50.8))
     (stroke (width 0) (type default))
   )
@@
     (stroke (width 0) (type default))
   )
-  (wire (pts (xy 69.85 48.26) (xy 76.2 48.26))
+  (wire (pts (xy 62.23 48.26) (xy 76.2 48.26))
     (stroke (width 0) (type default))
   )
@@
     (stroke (width 0) (type default))
   )
-  (bus (pts (xy 67.31 22.86) (xy 67.31 36.83))
+  (bus (pts (xy 59.69 22.86) (xy 59.69 36.83))
     (stroke (width 0) (type default))
   )
@@
     (stroke (width 0) (type default))
   )
-  (wire (pts (xy 69.85 104.14) (xy 76.2 104.14))
+  (wire (pts (xy 62.23 104.14) (xy 76.2 104.14))
     (stroke (width 0) (type default))
   )
@@
     (stroke (width 0) (type default))
   )
-  (wire (pts (xy 69.85 118.11) (xy 76.2 118.11))
-    (stroke (width 0) (type default))
-  )
   (wire (pts (xy 93.98 111.76) (xy 93.98 97.79))
     (stroke (width 0) (type default))
@@
     (stroke (width 0) (type default))
   )
-  (wire (pts (xy 69.85 34.29) (xy 76.2 34.29))
+  (wire (pts (xy 62.23 34.29) (xy 76.2 34.29))
     (stroke (width 0) (type default))
   )
@@
     (stroke (width 0) (type default))
   )
-  (wire (pts (xy 69.85 20.32) (xy 76.2 20.32))
-    (stroke (width 0) (type default))
-  )
-  (wire (pts (xy 69.85 76.2) (xy 76.2 76.2))
+  (wire (pts (xy 62.23 20.32) (xy 76.2 20.32))
+    (stroke (width 0) (type default))
+  )
+  (wire (pts (xy 62.23 76.2) (xy 76.2 76.2))
     (stroke (width 0) (type default))
   )
@@
     (stroke (width 0) (type default))
   )
-  (bus (pts (xy 67.31 78.74) (xy 67.31 92.71))
+  (bus (pts (xy 59.69 78.74) (xy 59.69 92.71))
     (stroke (width 0) (type default))
   )
@@
     (stroke (width 0) (type default))
   )
-  (bus (pts (xy 67.31 50.8) (xy 67.31 64.77))
+  (bus (pts (xy 59.69 50.8) (xy 59.69 64.77))
     (stroke (width 0) (type default))
   )
@@
     (stroke (width 0) (type default))
   )
-  (label "D2" (at 69.85 48.26 0) (fields_autoplaced)
-    (effects (font (size 1.27 1.27)) (justify left bottom))
-  )
-  (label "D7" (at 69.85 118.11 0) (fields_autoplaced)
-    (effects (font (size 1.27 1.27)) (justify left bottom))
-  )
-  (label "D0" (at 69.85 20.32 0) (fields_autoplaced)
-    (effects (font (size 1.27 1.27)) (justify left bottom))
-  )
-  (label "D1" (at 69.85 34.29 0) (fields_autoplaced)
-    (effects (font (size 1.27 1.27)) (justify left bottom))
-  )
-  (label "D5" (at 69.85 90.17 0) (fields_autoplaced)
+  (label "PixelOut2" (at 62.23 48.26 0) (fields_autoplaced)
+    (effects (font (size 1.27 1.27)) (justify left bottom))
+  )
+  (label "PixelOut4" (at 62.23 76.2 0) (fields_autoplaced)
     (effects (font (size 1.27 1.27)) (justify left bottom))
   )
@@
     (effects (font (size 1.27 1.27)) (justify left bottom))
   )
-  (label "D6" (at 69.85 104.14 0) (fields_autoplaced)
-    (effects (font (size 1.27 1.27)) (justify left bottom))
-  )
-  (label "D4" (at 69.85 76.2 0) (fields_autoplaced)
+  (label "PixelOut6" (at 62.23 104.14 0) (fields_autoplaced)
+    (effects (font (size 1.27 1.27)) (justify left bottom))
+  )
+  (label "PixelOut3" (at 62.23 62.23 0) (fields_autoplaced)
+    (effects (font (size 1.27 1.27)) (justify left bottom))
+  )
+  (label "PixelOut0" (at 62.23 20.32 0) (fields_autoplaced)
     (effects (font (size 1.27 1.27)) (justify left bottom))
   )
@@
     (effects (font (size 1.27 1.27)) (justify left bottom))
   )
-  (label "D3" (at 69.85 62.23 0) (fields_autoplaced)
+  (label "PixelOut7" (at 62.23 118.11 0) (fields_autoplaced)
+    (effects (font (size 1.27 1.27)) (justify left bottom))
+  )
+  (label "PixelOut1" (at 62.23 34.29 0) (fields_autoplaced)
+    (effects (font (size 1.27 1.27)) (justify left bottom))
+  )
+  (label "PixelOut5" (at 62.23 90.17 0) (fields_autoplaced)
     (effects (font (size 1.27 1.27)) (justify left bottom))
   )
@@
     (effects (font (size 1.27 1.27)) (justify left))
   )
-  (hierarchical_label "Pixel" (shape input) (at 67.31 120.65 180) (fields_autoplaced)
+  (hierarchical_label "PixelOut[0..7]" (shape input) (at 59.69 120.65 180) (fields_autoplaced)
     (effects (font (size 1.27 1.27)) (justify right))
   )

Commit message: work on DAC
Parts:
- added R1: 820, symbol Device:R
- added R10, R11, R9: 100, symbol Device:R
- added R2: 390, symbol Device:R
- added R3, R6: 1.8k, symbol Device:R
- added R4, R7: 910, symbol Device:R
- added R5, R8: 470, symbol Device:R
- U31: value 74LS08 -> 74LV08
Connections:
- net Blue: now also R1.2, R2.2, R9.1
- net Green: now also R10.1, R3.2, R4.2, R5.2
- net Red: now also R11.1, R6.2, R7.2, R8.2
- net at U30.6: now also R2.1
- net at U30.8: now also R3.1
- net at U30.11: now also R4.1
- net at U31.3: now also R5.1
- net at U31.6: now also R6.1
- net at U31.11: now also R8.1
- net at U31.8: now also R7.1
- net at U30.3: now also R1.1
- new net GND: R10.2, R11.2, R9.2
Other:
- moved on the sheet: U15C, U15D, U15E, U17A, U17B, U17C, U17D, U17E, U30C, U30D, U30E, U31A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

Commit message: work on main page layout
Connections:
- net ShowWhite is gone; now on net BlankWhite: U15.10, U15.13, U15.2, U15.5, U17.10, U17.13, U17.2, U17.5
- net ~{ShowBlack} renamed ~{BlankBlack}
Changed lines of the file:
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@@
     (stroke (width 0) (type default))
   )
-  (wire (pts (xy 60.96 146.05) (xy 73.66 146.05))
+  (wire (pts (xy 59.69 146.05) (xy 73.66 146.05))
     (stroke (width 0) (type default))
   )
@@
     (stroke (width 0) (type default))
   )
-  (wire (pts (xy 60.96 148.59) (xy 93.98 148.59))
+  (wire (pts (xy 59.69 148.59) (xy 93.98 148.59))
     (stroke (width 0) (type default))
   )
@@
     (effects (font (size 1.27 1.27)) (justify left bottom))
   )
-  (label "~{ShowBlack}" (at 60.96 148.59 0) (fields_autoplaced)
-    (effects (font (size 1.27 1.27)) (justify left bottom))
-  )
   (label "PixelOut6" (at 62.23 124.46 0) (fields_autoplaced)
     (effects (font (size 1.27 1.27)) (justify left bottom))
@@
   )
   (label "PixelOut0" (at 62.23 20.32 0) (fields_autoplaced)
-    (effects (font (size 1.27 1.27)) (justify left bottom))
-  )
-  (label "ShowWhite" (at 60.96 146.05 0) (fields_autoplaced)
     (effects (font (size 1.27 1.27)) (justify left bottom))
   )
@@
     (effects (font (size 1.27 1.27)) (justify left))
   )
-  (hierarchical_label "HBlank" (shape input) (at 40.64 138.43 180) (fields_autoplaced)
+  (hierarchical_label "~{BlankBlack}" (shape input) (at 59.69 148.59 180) (fields_autoplaced)
     (effects (font (size 1.27 1.27)) (justify right))
   )
-  (hierarchical_label "VBlank" (shape input) (at 40.64 140.97 180) (fields_autoplaced)
+  (hierarchical_label "BlankWhite" (shape input) (at 59.69 146.05 180) (fields_autoplaced)
     (effects (font (size 1.27 1.27)) (justify right))
   )
-  (hierarchical_label "BlankBlack" (shape input) (at 40.64 143.51 180) (fields_autoplaced)
-    (effects (font (size 1.27 1.27)) (justify right))
-  )
-  (hierarchical_label "BlankWhite" (shape input) (at 40.64 146.05 180) (fields_autoplaced)
-    (effects (font (size 1.27 1.27)) (justify right))
-  )

Commit message: misc fixes, start on pcb
Parts:
- removed unit 5 of U15
- removed unit 5 of U17
- removed unit 5 of U30
- removed unit 5 of U31
- R1, R10, R11, R2, R3, R4, R5, R6, R7, R8, R9: footprint (none) -> Resistor_SMD:R_1206_3216Metric_Pad1.30x1.75mm_HandSolder
- U15, U17, U30, U31: footprint (none) -> Package_SO:SOIC-14_3.9x8.7mm_P1.27mm
Other:
- moved on the sheet: R1, R10, R11, R2, R3, R4, R5, R6, R7, R8, R9, U15A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

Commit message: Work on layout/routing
Connections:
- net PixelOut0: now also U15.9; no longer U15.1
- net PixelOut2: now also U15.1; no longer U15.9
- net PixelOut4: now also U17.9; no longer U17.1
- net PixelOut6: now also U17.1; no longer U17.9
- net at U17.6: now also U31.9; no longer U31.4
- net at U30.4: now also U15.8; no longer U15.6
- net at U30.6: now also R1.1; no longer R2.1
- net at U15.11: now also U30.1; no longer U30.12
- net at U30.9: now also U15.6; no longer U15.8
- net at U30.8: now also R2.1; no longer R3.1
- net at U30.11: now also R3.1; no longer R4.1
- net at U17.11: now also U31.1; no longer U31.12
- net at R5.1: now also U31.6; no longer U31.3
- net at R6.1: now also U31.8; no longer U31.6
- net at U17.8: now also U31.4; no longer U31.9
- net at U17.3: now also U31.12; no longer U31.1
- net at U30.3: now also R4.1; no longer R1.1
- net at R8.1: now also U31.3; no longer U31.11
- net at R7.1: now also U31.11; no longer U31.8
- net at U15.3: now also U30.12; no longer U30.1
Other:
- moved on the sheet: U15A, U15C, U17A, U17C, U30A, U30B, U30C, U30D, U31A, U31B, U31C, U31D
